File: PCB/AI_EINK.sch (EAGLE design)
At the start: 127 parts, among them J3 524372471, Q1 SI1308EDL-T1-GE3, T1 MMUN2133LT1G, U1 TPS61090RSAR, U2 MC74VHC1G14DFT1G, U3 BQ27441DRZR-G1A, U4 BQ24075, U5 TLV74328, U6 TLV74315, U7 TPA2005D1DRB

Commit message: added mic interface and RFID
Parts:
- removed C28: 1uF, SparkFun:CAP1206
- removed C29: 10uF, SparkFun:CAP1206
- removed C41: 10uF, SparkFun-Capacitors:10UF-0603-6.3V-20%
- removed C42: 3.3nF, SparkFun-Capacitors:3.3NF-0603-100V-10%
- removed R16: 10K, SparkFun:RESISTOR0603-RES
- removed R17: 270R (ERJ-3EKF2700V), Resistor:R-US_CHIP-0603(1608-METRIC)
- removed R25: 150R (CR0805J150RP05Z), Resistor:R-US_CHIP-0603(1608-METRIC)
- removed R26, R27: 150K, SparkFun:RESISTOR0603-RES
- removed U7: TPA2005D1DRB, mike-temp:TPA2005D1DRB
- added ANT1: NFC_ANTENNA_25X15, microbuilder:NFC_ANTENNA_25X15
- added C45, C46, C56, C57, C65: 10uF, microbuilder:CAP_CERAMIC0805-NOOUTLINE
- added C47, C48, C49, C50, C51, C58: 0.1uF, microbuilder:CAP_CERAMIC0603_NO
- added C52, C53, C54, C55: 33pF, microbuilder:CAP_CERAMIC0603_NO
- added C63, C64: 100pF, microbuilder:CAP_CERAMIC0603_NO
- added C66: 2.2uF+, microbuilder:CAP_CERAMIC0805-NOOUTLINE
- added FB10, FB9: 120o, microbuilder:FERRITE-0805NO
- added FB3: Ferrite, microbuilder:FERRITE-0805NO
- added FB4: FERRITE, microbuilder:FERRITE-0805NO
- added IC3: WM8960, microbuilder:WM8960
- added LEFTMIC, RIGHTMIC: (no value), microbuilder:SPW2430HR5H-B
- added OSC2: ECS-3225MV, microbuilder:OSCILLATOR3.2X2.5
- added RF1: ST25DVXX_TSSOP, microbuilder:ST25DVXX_TSSOP
- C26: value 1uF -> 10uF; device SparkFun:CAP1206 -> microbuilder:CAP_CERAMIC0805-NOOUTLINE
- C27: value 1uF -> 0.1uF; device SparkFun:CAP1206 -> microbuilder:CAP_CERAMIC0603_NO
Connections:
- net MCLK renamed RFC_MCLK
- removed net AUDIO: C27.1, C41.2
- removed net IN+AMP: R26.2, U7.IN+
- removed net IN-AMP: R27.2, U7.IN-
- removed net N$33: C28.2, R27.1
- removed net N$34: LS1.P, U7.OUT+
- removed net N$35: LS1.N, U7.OUT-
- removed net SDN*: R16.1, U7.SHUTDOWN
- removed net SPEAKER: R17.1, RPI-CM1G$1.GPIO18
- new net AGND: IC3.AGND
- new net AUDIO_MCLK: IC3.MCLK, OSC2.OUT
- new net AVDD: C50.1, C51.1, C58.1, IC3.AVDD, LEFTMIC.VDD, RIGHTMIC.VDD
- new net GPO: RF1.GPO
- new net I2S_BCLK: IC3.BCLK, RPI-CM1G$1.GPIO21
- new net I2S_DIN: IC3.ADCDAT, RPI-CM1G$1.GPIO12
- new net I2S_DOUT: IC3.DACDAT, RPI-CM1G$1.GPIO16
- new net I2S_LRCLK: IC3.ADCLRC/GPIO1, IC3.DACLRC, RPI-CM1G$1.GPIO20
- new net LEFT_N: C64.1, FB10.P$2, LS1.N
- new net LEFT_P: C63.1, FB9.P$2, LS1.P
- new net LINPUT1: C56.2, IC3.LINPUT1
- new net MICBIAS: C46.1, C48.1, IC3.MICBIAS
- new net N$29: C52.1, FB3.P$1, RIGHTMIC.OUTPUT
- new net N$31: C53.1, FB4.P$1, LEFTMIC.OUTPUT
- new net N$36: C54.1, C57.1, FB3.P$2
- new net N$37: C55.1, C56.1, FB4.P$2
- new net N$40: FB9.P$1, IC3.SPK_LP
- new net N$41: FB10.P$1, IC3.SPK_LN
- new net RINPUT1: C57.2, IC3.RINPUT1
- new net VEH: RF1.V_EH
- new net VMID: C45.1, C47.1, IC3.VMID
- net 3.3V: now also C26.1, C27.1, C49.1, IC3.DBVDD, IC3.DCVDD, OSC2.INH, OSC2.VCC, RF1.VCC
- net 5.0V: now also C65.1, C66.1, IC3.SPKVDD1, IC3.SPKVDD2; no longer C26.1, C29.1, R16.2, U7.VDD
- net GND: now also C27.2, C45.2, C46.2, C47.2, C48.2, C49.2, C50.2, C51.2, C52.2, C53.2, C54.2, C55.2, C58.2, C63.2, C64.2, C65.2, C66.2, IC3.DGND, IC3.SPKGND1, IC3.SPKGND2, LEFTMIC.GND@1, LEFTMIC.GND@2, OSC2.GND, RF1.GND, RIGHTMIC.GND@1, RIGHTMIC.GND@2; no longer C28.1, C29.2, C42.1, R25.1, U7.GND@1, U7.GND@2, U7.GND@3, U7.GND@4, U7.GND@5
- net N$16: now also ANT1.2, RF1.AC0; no longer C41.1, C42.2, R17.2, R25.2
- net N$32: now also ANT1.1, RF1.AC1; no longer C27.2, R26.1
- net SCL: now also IC3.SCL, RF1.SCL
- net SDA: now also IC3.SDA, RF1.SDA
Other:
- note removed: "(SEE DATASHEET FOR VALUES)"
- note removed: "FOR HIGHER GAIN, CHANGE R1, R2"
- note removed: "USING THROUGH-HOLE PADS R1A, R2A"
- moved on the sheet: C26, C27

Commit message: A
Parts:
- removed R31: 100k, SparkFun-Resistors:100KOHM-1/10W-1%(0603)
- removed SJ2, SJ3, SJ4: JUMPER-PAD-2-NC_BY_TRACE, SparkFun-Passives:JUMPER-PAD-2-NC_BY_TRACE
- added BOOST_EN, COUNTER_CLR, GND10, GND11, GND29, PULSE_555: TEST-POINT3, SparkFun-Connectors:TEST-POINT3
- added C28: 1uF, Capacitor:C_CHIP-0603(1608-METRIC)
- added C29, C41: 0.1uF, Capacitor:C-US_CHIP-0603(1608-METRIC)
- added C42: 0.1uF, microbuilder:CAP_CERAMIC0805_10MGAP
- added J1: BM04B-GHS-TBT(LF)(SN)(N), BM04B-GHS-TBT_LF__SN__N_:BM04B-GHS-TBT(LF)(SN)(N)
- added OV5674: DF30FC-24DS-0.4V(82)CONN_DF30FC-24DS-0.4V(82)_HIR, 2024-03-07_05-07-01_Library:DF30FC-24DS-0.4V(82)CONN_DF30FC-24DS-0.4V(82)_HIR
- added Q3: 2A/20V/150mΩ, SparkFun-DiscreteSemi:MOSFET_PCH_DUAL-DMP2240UDM
- added R16: 280k, Resistor:R-US_CHIP-0603(1608-METRIC)
- added R17, R25, R26, R27: 10k, Resistor:R-US_CHIP-0603(1608-METRIC)
- added R30: 36k, Resistor:R-US_CHIP-0603(1608-METRIC)
- added SW1: (no value), adafruit:SWITCH_PUSHBUTTONSOFTTOUCHSMD_SJ
- added U7: NE555DR, IC:NE555DR
- added U8: SN74LV4040ARGYRRGY16_2P55X2P05, 2024-03-07_02-24-03_Library:SN74LV4040ARGYRRGY16_2P55X2P05
- added U9: EMC2301-1-ACZL-TRMSOP8_MC_MCH-L, 2024-03-07_04-01-04_Library:EMC2301-1-ACZL-TRMSOP8_MC_MCH-L
- C16: value 0.1uF -> 1uF
- C18: value 0.1uF -> 4.7uF
- R19: value 590 -> 10K; device SparkFun-Passives:RESISTOR0603-RES -> Resistor:R-US_CHIP-0603(1608-METRIC); PROD_ID RES-13217 -> (none)
- R21: value 1.1k -> 10k; device SparkFun-Passives:RESISTOR0603-RES -> Resistor:R-US_CHIP-0603(1608-METRIC); PROD_ID RES-10447 -> (none)
Connections:
- removed net N$24: R31.2, S1.O
- removed net N$26: R21.1, SJ4.1
- removed net N$27: R19.1, SJ3.1
- removed net N$30: C10.2, C11.2, C12.2, C9.2, J3.8
- removed net SYSOFF: S1.P, U4.SYSOFF
- removed net TMR: SJ2.2, U4.TMR
- new net BOOST_EN: BOOST_EN.1, R13.1, S1.P, U8.QD
- new net COUNTER_CLR: COUNTER_CLR.1, Q3G$1.D, R19.2, U8.CLR, U8.QF
- new net FAN_PWM: J1.1, U9.PWM
- new net POWER_OFF_MCU: Q3G$1.G, RPI-CM1G$1.GPIO25
- new net POWER_SWITCH_N: Q3G1.G, R17.2, RPI-CM1G$1.GPIO7, SW1.P$2
- new net PULSE_555: PULSE_555.1, U7.OUT, U8.CLK
- new net PWM_FAN: RPI-CM1G$1.GPIO14
- new net TACH: J1.2, R30.1, U9.TACH
- new net TRIG: C28.1, R16.1, U7.THRES, U7.TRIG
- new net V_OUT: Q3G$1.S, Q3G1.S, S1.O, SW1.P$1, U8.VCC
- net 3.3V: now also R26.2, R27.2, R30.2, U9.VDD
- net 5.0V: now also C42.1, J1.3
- net GDR: now also Q1.G, R11.2
- net GND: now also C10.2, C11.2, C12.2, C13.2, C14.2, C15.2, C28.2, C29.2, C41.2, C42.2, C9.2, GND10.1, GND11.1, GND29.1, J1.4, J1.SHIELD, J3.8, R17.1, R19.1, U4.SYSOFF, U4.TMR, U7.GND, U8.GND, U9.GND; no longer R19.2, R21.2, SJ2.1
- net ILIM: no longer SJ4.2
- net ISET: no longer SJ3.2
- net N$18: now also Q3G1.D, R16.2, U7.DISCH, U7.RESET, U7.VCC; no longer C13.2, C14.2, C15.2
- net N$20: now also R21.2, R26.1, VR1.A; no longer Q1.S, R9.2
- net N$22: now also R25.2, R27.1, VR1.B; no longer Q1.G, R11.2
- net RESE: now also Q1.S, R9.2
- net ROT1: now also C41.1, R25.1; no longer VR1.B
- net ROT2: now also C29.1, R21.1; no longer VR1.A
- net SCL: now also U9.SMCLK
- net SDA: now also U9.SMDATA
- net VOUT: no longer R13.1
- net V_BATT: no longer R31.1
Other:
- moved on the sheet: R19, R21, S1, VR1

Commit message: a
Connections:
- net SCL: now also RPI-CM1G$1.GPIO3; no longer RPI-CM1G$1.GPIO2
- net SDA: now also RPI-CM1G$1.GPIO2; no longer RPI-CM1G$1.GPIO3
Changed lines of the file:
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@@
-</segment>
-<segment>
-<pinref part="RPI-CM1" gate="G$1" pin="GPIO3"/>
-<wire x1="91.44" y1="76.2" x2="99.06" y2="76.2" width="0.1524" layer="91"/>
-<label x="93.98" y="76.2" size="1.778" layer="95"/>
 </segment>
 <segment>
@@
 <label x="449.58" y="144.78" size="1.778" layer="95"/>
 </segment>
+<segment>
+<pinref part="RPI-CM1" gate="G$1" pin="GPIO2"/>
+<wire x1="91.44" y1="73.66" x2="96.52" y2="73.66" width="0.1524" layer="91"/>
+<label x="91.44" y="73.66" size="1.778" layer="95"/>
+</segment>
 </net>
 <net name="SCL" class="0">
@@
 <wire x1="454.66" y1="241.3" x2="441.96" y2="241.3" width="0.1524" layer="91"/>
 <label x="441.96" y="241.3" size="1.27" layer="95" font="vector" rot="R180" xref="yes"/>
-</segment>
-<segment>
-<pinref part="RPI-CM1" gate="G$1" pin="GPIO2"/>
-<wire x1="91.44" y1="73.66" x2="99.06" y2="73.66" width="0.1524" layer="91"/>
-<label x="93.98" y="73.66" size="1.778" layer="95"/>
 </segment>
 <segment>
@@
 <label x="449.58" y="154.94" size="1.778" layer="95"/>
 </segment>
+<segment>
+<pinref part="RPI-CM1" gate="G$1" pin="GPIO3"/>
+<wire x1="91.44" y1="76.2" x2="96.52" y2="76.2" width="0.1524" layer="91"/>
+<label x="91.44" y="76.2" size="1.778" layer="95"/>
+</segment>
 </net>

Commit message: a
Parts:
- removed BOOST_EN, COUNTER_CLR, GND10, GND11, GND29, PULSE_555: TEST-POINT3, SparkFun-Connectors:TEST-POINT3
- removed C40: 1nF, SparkFun-Capacitors:1.0NF/1000PF-0603-50V-10%
- removed C41: 0.1uF, Capacitor:C-US_CHIP-0603(1608-METRIC)
- removed C51: 0.1uF, microbuilder:CAP_CERAMIC0603_NO
- removed C53, C55: 33pF, microbuilder:CAP_CERAMIC0603_NO
- removed C56: 10uF, microbuilder:CAP_CERAMIC0805-NOOUTLINE
- removed FB4: FERRITE, microbuilder:FERRITE-0805NO
- removed FL1, FL2: BLM18HE152SN1D, BLM18HE152SN1D:BLM18HE152SN1D
- removed LEFTMIC, RIGHTMIC: (no value), microbuilder:SPW2430HR5H-B
- removed OV5647: DF30FC-24DP-0.4V(81), DF30FC-24DP-0.4V_81_:DF30FC-24DP-0.4V(81)
- removed Q3: 2A/20V/150mΩ, SparkFun-DiscreteSemi:MOSFET_PCH_DUAL-DMP2240UDM
- removed R19: 10K, Resistor:R-US_CHIP-0603(1608-METRIC)
- removed R21, R25, R26, R27: 10k, Resistor:R-US_CHIP-0603(1608-METRIC)
- removed S2: FSMRA4JH04, FSMRA4JH04:FSMRA4JH04
- removed SJ5: JUMPER-PAD-3-2OF3_NC_BY_TRACE_SMALL, SparkFun-Passives:JUMPER-PAD-3-2OF3_NC_BY_TRACE_SMALL
- removed SW1: (no value), adafruit:SWITCH_PUSHBUTTONSOFTTOUCHSMD_SJ
- removed U8: SN74LV4040ARGYRRGY16_2P55X2P05, 2024-03-07_02-24-03_Library:SN74LV4040ARGYRRGY16_2P55X2P05
- removed VR1: EC10E1220501, EC10E1220501:EC10E1220501
- added B_D, B_S, B_U: FSMRA4JH04, FSMRA4JH04:FSMRA4JH04
- added C2040: RP2040TR13QFN56_7X7_RPI, 2024-03-10_01-36-20_Library:RP2040TR13QFN56_7X7_RPI
- added C43, C44, C67, C69, C70, C71, C72, C73, C74, C77, C78, C81: 0.1uF, Capacitor:C_CHIP-0603(1608-METRIC)
- added C59, C60, C61, C62, C68, C79, C80: 10uF, Capacitor:C_CHIP-0603(1608-METRIC)
- added C75, C76: 1.0uF, Capacitor:C_CHIP-0603(1608-METRIC)
- added C82, C83: 15p, Capacitor:C_CHIP-0603(1608-METRIC)
- added D7: PMIC, SparkFun-LED:LED-RED0603
- added FB2, FB5: Ferrite, microbuilder:FERRITE0805
- added FL3, FL4, FL5: BLM18HE152SN1D, BLM18HE152SN1D:BLM18HE152SN1D
- added GND34, USB_BOOT_N: TEST-POINT3, SparkFun-Connectors:TEST-POINT3
- added Q2: 2.5A/30V, User-Submitted:MOSFET-PCHANNELDMG2307L
- added R31, R32: 27, resistor:R-US_R0603
- added R34, R35: 1k, resistor:R-US_R0603
- added R36, R37: 200K, resistor:R-US_R0603
- added SJ2, SJ3: JUMPER-PAD-3-2OF3_NC_BY_TRACE_SMALL, SparkFun-Passives:JUMPER-PAD-3-2OF3_NC_BY_TRACE_SMALL
- added SPI_FLASH_SAM: W25Q128JVBIQTFBGA_128JVBIQ_WIN, 2024-03-10_02-04-46_Library:W25Q128JVBIQTFBGA_128JVBIQ_WIN
- added U10, U11: AP2112-3.3K, microbuilder:VREG_SOT23-5
- added U12: SPU0410LR5H-QB, SPU0410LR5H-QB:SPU0410LR5H-QB
- added Y1: ABM8-272-T3, ABM8-272-T3:ABM8-272-T3
- C1, C2, C24, C26, C3, C31, C32, C33, C34, C35, C45, C46, C57, C65, C66, C7: device microbuilder:CAP_CERAMIC0805-NOOUTLINE -> Capacitor:C_CHIP-0603(1608-METRIC)
- C16, C17, C18, C4, C42: device microbuilder:CAP_CERAMIC0805_10MGAP -> Capacitor:C_CHIP-0603(1608-METRIC)
- C19: device SparkFun-Capacitors:1.0UF-16V-10%(0603) -> Capacitor:C_CHIP-0603(1608-METRIC)
- C20: device SparkFun-Capacitors:CAP0603-CAP -> Capacitor:C_CHIP-0603(1608-METRIC)
- C21, C23: device SparkFun-Capacitors:10UF10V10%(0805) -> Capacitor:C_CHIP-0603(1608-METRIC)
- C22: device SparkFun-Capacitors:1.0UF50V10%(1206) -> Capacitor:C_CHIP-0603(1608-METRIC)
- C25: value 0.1uF -> 1.0uF; device microbuilder:CAP_CERAMIC0603_NO -> Capacitor:C_CHIP-0603(1608-METRIC)
- C27, C30, C47, C48, C49, C50, C52, C54, C58, C63, C64: device microbuilder:CAP_CERAMIC0603_NO -> Capacitor:C_CHIP-0603(1608-METRIC)
- C28: value 1uF -> 10uF
- C29: value 0.1uF -> 10uF; device Capacitor:C-US_CHIP-0603(1608-METRIC) -> Capacitor:C_CHIP-0603(1608-METRIC)
- C36, C37, C38, C39: value 1nF -> 10uF; device SparkFun-Capacitors:1.0NF/1000PF-0603-50V-10% -> Capacitor:C_CHIP-0603(1608-METRIC)
- J2: value (none) -> C393939
- R1, R2: device microbuilder:RESISTOR_0805MP -> resistor:R-US_R0603
- R10, R8: device rcl:R-US_R0603 -> resistor:R-US_R0603
- R11, R17, R30, R9: device Resistor:R-US_CHIP-0603(1608-METRIC) -> resistor:R-US_R0603
- R13, R20, R3, R4, R5: device microbuilder:RESISTOR0805_NOOUTLINE -> resistor:R-US_R0603
- R14: value 10K -> 1K; device microbuilder:RESISTOR_0603_NOOUT -> resistor:R-US_R0603
- R15, R18: device SparkFun-Resistors:4.7KOHM-1/10W-1%(0603) -> resistor:R-US_R0603
- R16: value 280k -> 10k; device Resistor:R-US_CHIP-0603(1608-METRIC) -> resistor:R-US_R0603
- R22: device SparkFun-Resistors:180OHM1/10W1%(0603) -> resistor:R-US_R0603
- R23: device SparkFun-Resistors:1KOHM-1/10W-1%(0603) -> resistor:R-US_R0603
- R24: device SparkFun-Resistors:100KOHM-1/10W-1%(0603) -> resistor:R-US_R0603
- R28: value 1k -> 10k; device rcl:R-US_R0603 -> resistor:R-US_R0603
- R29, R33: device SparkFun-Resistors:10KOHM-1/10W-1%(0603)0603 -> resistor:R-US_R0603
- R6, R7: device SparkFun-Passives:RESISTOR0603-RES -> resistor:R-US_R0603
- U7: value NE555DR -> TLV74318PDBVRDBV0005A_L; device IC:NE555DR -> 2024-03-10_03-34-55_Library:TLV74318PDBVRDBV0005A_L
Connections:
- removed net !PGOOD!: SJ5.1, U4.!PGOOD!
- removed net BUTTON: RPI-CM1G$1.GPIO26, S2.NO
- removed net COUNTER_CLR: COUNTER_CLR.1, Q3G$1.D, R19.2, U8.CLR, U8.QF
- removed net LINPUT1: C56.2, IC3.LINPUT1
- removed net N$20: R21.2, R26.1, VR1.A
- removed net N$22: R25.2, R27.1, VR1.B
- removed net N$28: R23.2, SJ5.2
- removed net N$31: C53.1, FB4.P$1, LEFTMIC.OUTPUT
- removed net N$37: C55.1, C56.1, FB4.P$2
- removed net POWER_OFF_MCU: Q3G$1.G, RPI-CM1G$1.GPIO25
- removed net POWER_SWITCH_N: Q3G1.G, R17.2, RPI-CM1G$1.GPIO7, SW1.P$2
- removed net PULSE_555: PULSE_555.1, U7.OUT, U8.CLK
- removed net PWM_FAN: RPI-CM1G$1.GPIO14
- removed net ROT1: C41.1, R25.1, RPI-CM1G$1.GPIO22
- removed net ROT2: C29.1, R21.1, RPI-CM1G$1.GPIO17
- removed net TRIG: C28.1, R16.1, U7.THRES, U7.TRIG
- removed net V_OUT: Q3G$1.S, Q3G1.S, S1.O, SW1.P$1, U8.VCC
- new net AF_EN: OV5674.18
- new net BUTTON_D: B_D.NO, C2040.GPIO18
- new net BUTTON_S: B_S.NO, C2040.GPIO16
- new net BUTTON_U: B_U.NO, C2040.GPIO17
- new net N$24: R34.2, USB_BOOT_N.1
- new net N$26: C83.2, R35.2, Y1.CRYSTAL_2
- new net N$27: R37.1, S1.S
- new net OUT: C62.1, C69.1, FB2.P$2, U10.OUT
- new net PI_1V8: RPI-CM1G$1.CM4_1.8V(OUTPUT)@88, RPI-CM1G$1.CM4_1.8V(OUTPUT)@90
- new net PWDN: OV5674.19, SJ3.2
- new net RESET: OV5674.22, SJ2.2
- new net SAM_1V1: C2040.DVDD, C2040.DVDD_2, C2040.VREG_VOUT, C76.1, C77.1, C78.1
- new net SAM_3V3: B_D.COM, B_S.COM, B_U.COM, C2040.ADC_AVDD, C2040.IOVDD, C2040.IOVDD_2, C2040.IOVDD_3, C2040.IOVDD_4, C2040.IOVDD_5, C2040.IOVDD_6, C2040.USB_VDD, C2040.VREG_VIN, C43.1, C44.1, C70.1, C71.1, C72.1, C73.1, C74.1, C75.1, C80.1, C81.1, D7.A, R16.2, R17.2, R28.2, SPI_FLASH_SAM.VCC, U11.OUT
- new net SAM_GPIO0: C2040.GPIO0
- new net SAM_GPIO1: C2040.GPIO1
- new net SAM_GPIO10: C2040.GPIO10
- new net SAM_GPIO11: C2040.GPIO11
- new net SAM_GPIO12: C2040.GPIO12
- new net SAM_GPIO13: C2040.GPIO13
- new net SAM_GPIO14: C2040.GPIO14
- new net SAM_GPIO15: C2040.GPIO15
- new net SAM_GPIO2: C2040.GPIO2
- new net SAM_GPIO22: C2040.GPIO22
- new net SAM_GPIO23: C2040.GPIO23
- new net SAM_GPIO24: C2040.GPIO24
- new net SAM_GPIO25: C2040.GPIO25
- new net SAM_GPIO26/ADC0: C2040.GPIO26/ADC0
- new net SAM_GPIO27/ADC1: C2040.GPIO27/ADC1
- new net SAM_GPIO28/ADC2: C2040.GPIO28/ADC2
- new net SAM_GPIO29/ADC3: C2040.GPIO29/ADC3
- new net SAM_GPIO3: C2040.GPIO3
- new net SAM_GPIO4: C2040.GPIO4
- new net SAM_GPIO5: C2040.GPIO5
- new net SAM_GPIO6: C2040.GPIO6
- new net SAM_GPIO7: C2040.GPIO7
- new net SAM_GPIO8: C2040.GPIO8
- new net SAM_GPIO9: C2040.GPIO9
- new net SAM_QSPI_SCLK: C2040.QSPI_SCLK, SPI_FLASH_SAM.CLK
- new net SAM_QSPI_SCN: C2040.QSPI_SCN, R34.1, SPI_FLASH_SAM./CS
- new net SAM_QSPI_SD0: C2040.QSPI_SD0, SPI_FLASH_SAM.DI_(IO0)
- new net SAM_QSPI_SD1: C2040.QSPI_SD1, SPI_FLASH_SAM.DO_(IO1)
- new net SAM_QSPI_SD2: C2040.QSPI_SD2, SPI_FLASH_SAM./WP_(IO2)
- new net SAM_QSPI_SD3: C2040.QSPI_SD3, SPI_FLASH_SAM./HOLD_(IO3)
- new net SAM_RUN: C2040.RUN
- new net SAM_SWCLK: C2040.SWCLK
- new net SAM_SWD: C2040.SWD
- new net SAM_USB_DM: C2040.USB_DM, R32.2
- new net SAM_USB_DP: C2040.USB_DP, R31.2
- new net SAM_XIN: C2040.XIN, C82.1, Y1.CRYSTAL_1
- new net SAM_XOUT: C2040.XOUT, R35.1
- new net STROBE: OV5674.20
- new net SYS_POW_SAM: C2040.GPIO21, Q2.G
- net 1.5V: now also FL3.1; no longer FL2.1
- net 1.8V: now also C25.1, C28.1, C29.1, FL4.1, SJ2.3, SJ3.1, U7.OUT; no longer RPI-CM1G$1.CM4_1.8V(OUTPUT)@88, RPI-CM1G$1.CM4_1.8V(OUTPUT)@90
- net 2.8V: now also FL5.1; no longer C38.1, FL1.1, OV5647.PIN19
- net 3.3V: now also C36.1, C37.1, C38.1, C39.1, U7.EN, U7.IN; no longer C25.1, R26.2, R27.2, R28.2, S2.COM
- net 5.0V: now also C59.1, C60.1, C61.1, U10.EN, U10.IN
- net AGND: now also C67.2, C68.2, FB5.P$1
- net AVDD: now also C67.1, C68.1, FB2.P$1, U12.VDD; no longer C51.1, LEFTMIC.VDD, RIGHTMIC.VDD
- net BOOST_EN: now also Q2.D, R36.1; no longer BOOST_EN.1, U8.QD
- net CAM0_C_N: now also OV5674.8; no longer OV5647.PIN8
- net CAM0_C_P: now also OV5674.9; no longer OV5647.PIN7
- net CAM0_D0_N: now also OV5674.2; no longer OV5647.PIN10
- net CAM0_D0_P: now also OV5674.3; no longer OV5647.PIN9
- net CAM0_D1_N: now also OV5674.5; no longer OV5647.PIN6
- net CAM0_D1_P: now also OV5674.6; no longer OV5647.PIN5
- net EINK_BUSY: now also RPI-CM1G$1.GPIO5; no longer RPI-CM1G$1.GPIO19
- net GND: now also C2040.GND, C2040.TESTEN, C43.2, C44.2, C59.2, C60.2, C61.2, C62.2, C69.2, C70.2, C71.2, C72.2, C73.2, C74.2, C75.2, C76.2, C77.2, C78.2, C79.2, C80.2, C81.2, C82.2, C83.1, FB5.P$2, GND34.1, OV5674.1, OV5674.10, OV5674.12, OV5674.21, OV5674.4, OV5674.7, R16.1, R23.2, R36.2, R37.2, SJ2.1, SJ3.3, SPI_FLASH_SAM.GND, U10.GND, U11.GND, U12.GND, Y1.GND_1, Y1.GND_2; no longer C40.2, C41.2, C51.2, C53.2, C55.2, GND10.1, GND11.1, GND29.1, LEFTMIC.GND@1, LEFTMIC.GND@2, OV5647.PIN13, OV5647.PIN15, OV5647.PIN17, R19.1, RIGHTMIC.GND@1, RIGHTMIC.GND@2, S1.S, SJ5.3, U8.GND, VR1.C
- net I2S_BCLK: now also RPI-CM1G$1.GPIO18; no longer RPI-CM1G$1.GPIO21
- net I2S_DIN: now also RPI-CM1G$1.GPIO20; no longer RPI-CM1G$1.GPIO12
- net I2S_DOUT: now also RPI-CM1G$1.GPIO21; no longer RPI-CM1G$1.GPIO16
- net I2S_LRCLK: now also RPI-CM1G$1.GPIO19; no longer RPI-CM1G$1.GPIO20
- net N$10: now also FL4.2, OV5674.15; no longer OV5647.PIN24, R14.1
- net N$13: now also FL3.2, OV5674.13, OV5674.14; no longer C39.1, C40.1, FL2.2, OV5647.PIN20
- net N$18: now also D7.C, R14.1; no longer Q3G1.D, R16.2, U7.DISCH, U7.RESET, U7.VCC
- net N$29: now also U12.OUTPUT; no longer RIGHTMIC.OUTPUT
- net N$8: now also FL5.2, OV5674.16, OV5674.17; no longer C36.1, C37.1, FL1.2, OV5647.PIN18
- net RFC_MCLK: now also OV5674.11; no longer OV5647.PIN14
- net SCL: now also OV5674.23; no longer OV5647.PIN11
- net SDA: now also OV5674.24; no longer OV5647.PIN12
- net USB_N: now also R32.1
- net USB_P: now also R31.1
- net VOUT: now also C79.1, Q2.S, S1.O, U11.EN, U11.IN
Other:
- moved on the sheet: ANT1, C1, C16, C17, C18, C19, C2, C20, C21, C22, C23, C24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

Commit message: a
Parts:
- removed B_D, B_S, B_U: FSMRA4JH04, FSMRA4JH04:FSMRA4JH04
- removed Q2: 2.5A/30V, User-Submitted:MOSFET-PCHANNELDMG2307L
- removed RF1: ST25DVXX_TSSOP, microbuilder:ST25DVXX_TSSOP
- added BUD, BUP, BUS: EVQ-P7A01P, EVQ-P7A01P:EVQ-P7A01P
- added Q3: NMOS_C7465427, Transistor:NMOSFETSOT23-GSD
- added U8: ST25DV64K-IER6S3SOIC_IER6S3_STM, 2024-03-10_23-40-44_Library:ST25DV64K-IER6S3SOIC_IER6S3_STM
- GND, GND13, GND22, GND25, GND26, GND27, GND34, RPIBOOT, RPIBOOT1, RPIBOOT2, RPIBOOT3, RPIBOOT4, USB_BOOT_N: value TEST-POINT3 -> DNP
- JP6: value (none) -> S2B-PH-SM4-TB
- S1: value (none) -> C963206
- SJ1, SJ6: value JUMPER-PAD-2-NC_BY_TRACE -> DNP
- SJ2, SJ3: value JUMPER-PAD-3-2OF3_NC_BY_TRACE_SMALL -> DNP
Connections:
- net 3.3V: now also U8.VCC; no longer RF1.VCC
- net BOOST_EN: now also Q3.D, R36.2; no longer Q2.D, R36.1
- net BUTTON_D: now also BUD.2; no longer B_D.NO
- net BUTTON_S: now also BUS.2; no longer B_S.NO
- net BUTTON_U: now also BUP.2; no longer B_U.NO
- net GND: now also Q3.S, U8.VSS; no longer R36.2, RF1.GND
- net GPO: now also U8.GPO; no longer RF1.GPO
- net N$16: now also U8.AC0; no longer RF1.AC0
- net N$32: now also U8.AC1; no longer RF1.AC1
- net SAM_3V3: now also BUD.1, BUP.1, BUS.1; no longer B_D.COM, B_S.COM, B_U.COM
- net SCL: now also U8.SCL; no longer RF1.SCL
- net SDA: now also U8.SDA; no longer RF1.SDA
- net SYS_POW_SAM: now also Q3.G; no longer Q2.G
- net VEH: now also U8.V_EH; no longer RF1.V_EH
- net VOUT: now also R36.1; no longer Q2.S
Other:
- moved on the sheet: ANT1, R36

Commit message: PCB
Parts:
- added C40, C41, C51, C53: 10uF, Capacitor:C_CHIP-0603(1608-METRIC)
- C22: value 1.0uF -> 10uF
Connections:
- net GND: now also C40.2, C41.2, C51.2, C53.2
- net VBUS: now also C53.1
- net V_BATT: now also C40.1, C41.1, C51.1
Other:
- moved on the sheet: C22, C23

Commit message: pcb before downsize
Parts:
- U1: value TPS61090RSAR -> TPS61092RSAR
Connections:
- new net N$20: RPI-CM1G$1.GPIO16
- new net N$22: RPI-CM1G$1.GPIO25
- new net N$28: RPI-CM1G$1.GPIO14
Changed lines of the file:
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@@
 <parts>
 <part name="RPI-CM1" library="RPI-CM4" deviceset="RPI-CM4" device="" value="DF40C-100DS-0.4V(51)"/>
-<part name="U1" library="microbuilder" deviceset="VREG_TPS6103X" device="" value="TPS61090RSAR"/>
+<part name="U1" library="microbuilder" deviceset="VREG_TPS6103X" device="" value="TPS61092RSAR"/>
 <part name="L1" library="microbuilder" deviceset="INDUCTOR" device="TDK_VLC5045" value="6.8uH"/>
 <part name="U$1" library="microbuilder" deviceset="GND" device=""/>
@@
 </segment>
 </net>
+<net name="N$20" class="0">
+<segment>
+<pinref part="RPI-CM1" gate="G$1" pin="GPIO16"/>
+<wire x1="30.48" y1="109.22" x2="5.08" y2="109.22" width="0.1524" layer="91"/>
+</segment>
+</net>
+<net name="N$22" class="0">
+<segment>
+<pinref part="RPI-CM1" gate="G$1" pin="GPIO25"/>
+<wire x1="30.48" y1="93.98" x2="5.08" y2="93.98" width="0.1524" layer="91"/>
+</segment>
+</net>
+<net name="N$28" class="0">
+<segment>
+<pinref part="RPI-CM1" gate="G$1" pin="GPIO14"/>
+<wire x1="30.48" y1="76.2" x2="5.08" y2="76.2" width="0.1524" layer="91"/>
+</segment>
+</net>
