File: PCB/AI_EINK.sch (EAGLE design)
At the start: 172 parts, among them IC3 WM8960, J1 BM04B-GHS-TBT(LF)(SN)(N), J2 C393939, Q1 SI1308EDL-T1-GE3, Q2 DMG2307L, Q3 NMOS_C7465427, T1 MMUN2133LT1G, U1 TPS61092RSAR, U10 AP2112-3.3K, U11 AP2112-3.3K, U12 C233266, U13 TPD4EUSB30DQARDQA10, U14 OPA344, U2 MC74VHC1G14DFT1G, U3 BQ27441DRZR-G1A, U4 BQ24075, U5 MC74VHC1G14DFT1G OR C66196, U6 W25Q128JVSIQSOIC_128JVSIQ_WIN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, U8 MC74VHC1G14DFT1G, U9 EMC2301-1-ACZL-TRMSOP8_MC_MCH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, Y1 ABM8-272-T3

Commit message: pcb
Parts:
- removed L2: ASPI-0403S-100M-T, ASPI-0403S-100M-T:ASPI-0403S-100M-T
- added L3: FNR5012S100MT 10uH, LQH5BPN2R2NT0L:LQH5BPN2R2NT0L
- added RPIBOOT3: DNP, SparkFun-Connectors:TEST-POINT3
- CAMERA: value 524372271CON_524372271_MOL -> C262642
- L1: value 6.8uH -> 6.8uH C36410
- LED2: value 5VBOOST -> LED_RED; device microbuilder:LED0805_NOOUTLINE -> LED:CHIP-ROUND-R_0603
- LOW_BATT: value XL-2012VRC -> LED_RED; device microbuilder:LED0805_NOOUTLINE -> LED:CHIP-ROUND-R_0603
Connections:
- net 3V3_EINK: now also L3.1; no longer L2.1
- net EXT_VCC_PCIE: now also RPIBOOT3.1
- net N$23: now also L3.2; no longer L2.2
Changed lines of the file:
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@@
 <part name="RPI-CM1" library="RPI-CM4" deviceset="RPI-CM4" device="" value="DF40C-100DS-0.4V(51)"/>
 <part name="U1" library="microbuilder" deviceset="VREG_TPS6103X" device="" value="TPS61092RSAR"/>
-<part name="L1" library="microbuilder" deviceset="INDUCTOR" device="TDK_VLC5045" value="6.8uH"/>
+<part name="L1" library="microbuilder" deviceset="INDUCTOR" device="TDK_VLC5045" value="6.8uH C36410"/>
 <part name="U$1" library="microbuilder" deviceset="GND" device=""/>
 <part name="U$2" library="microbuilder" deviceset="GND" device=""/>
@@
 <part name="C2" library="Capacitor" library_urn="urn:adsk.eagle:library:16290819" deviceset="C" device="CHIP-0402(1005-METRIC)" package3d_urn="urn:adsk.eagle:package:16290895/5" technology="_" value="2.2uF"/>
 <part name="U$7" library="microbuilder" deviceset="5.0V" device=""/>
-<part name="LOW_BATT" library="microbuilder" deviceset="LED" device="0805_NOOUTLINE" value="XL-2012VRC"/>
+<part name="LOW_BATT" library="LED" library_urn="urn:adsk.eagle:library:22900745" deviceset="CHIP-ROUND-R" device="_0603" package3d_urn="urn:adsk.eagle:package:24294800/1" value="LED_RED"/>
 <part name="R20" library="Resistor" library_urn="urn:adsk.eagle:library:16378527" deviceset="R-US" device="CHIP-0402(1005-METRIC)" package3d_urn="urn:adsk.eagle:package:16378568/5" technology="_" value="1K"/>
-<part name="LED2" library="microbuilder" deviceset="LED" device="0805_NOOUTLINE" value="5VBOOST"/>
+<part name="LED2" library="LED" library_urn="urn:adsk.eagle:library:22900745" deviceset="CHIP-ROUND-R" device="_0603" package3d_urn="urn:adsk.eagle:package:24294800/1" value="LED_RED"/>
 <part name="R5" library="Resistor" library_urn="urn:adsk.eagle:library:16378527" deviceset="R-US" device="CHIP-0402(1005-METRIC)" package3d_urn="urn:adsk.eagle:package:16378568/5" technology="_" value="1K"/>
 <part name="R13" library="Resistor" library_urn="urn:adsk.eagle:library:16378527" deviceset="R-US" device="CHIP-0402(1005-METRIC)" package3d_urn="urn:adsk.eagle:package:16378568/5" technology="_" value="200K"/>
@@
 <part name="U$83" library="microbuilder" deviceset="GND" device=""/>
 <part name="U$84" library="microbuilder" deviceset="GND" device=""/>
-<part name="L2" library="ASPI-0403S-100M-T" deviceset="ASPI-0403S-100M-T" device=""/>
 <part name="U$85" library="microbuilder" deviceset="GND" device=""/>
 <part name="U$86" library="microbuilder" deviceset="GND" device=""/>
@@
 <part name="GND10" library="supply1" deviceset="GND" device=""/>
 <part name="JOY_STICK" library="BM04B-GHS-TBT_LF__SN__N_" deviceset="BM04B-GHS-TBT(LF)(SN)(N)" device=""/>
-<part name="CAMERA" library="2024-03-29_02-21-27_Library" deviceset="524372271" device="CON_524372271_MOL"/>
+<part name="CAMERA" library="2024-03-29_02-21-27_Library" deviceset="524372271" device="CON_524372271_MOL" value="C262642"/>
 <part name="GND11" library="SparkFun-Aesthetics" deviceset="GND" device=""/>
 <part name="Q2" library="DMG2307L" deviceset="DMG2307L" device="" value="DMG2307L"/>
@@
 <part name="R43" library="Resistor" library_urn="urn:adsk.eagle:library:16378527" deviceset="R-US" device="CHIP-0402(1005-METRIC)" package3d_urn="urn:adsk.eagle:package:16378568/5" technology="_" value="10K"/>
 <part name="R44" library="Resistor" library_urn="urn:adsk.eagle:library:16378527" deviceset="R-US" device="CHIP-0402(1005-METRIC)" package3d_urn="urn:adsk.eagle:package:16378568/5" technology="_" value="6.57k"/>
+<part name="RPIBOOT3" library="SparkFun-Connectors" deviceset="TEST-POINT" device="3" value="DNP"/>
+<part name="L3" library="LQH5BPN2R2NT0L" deviceset="LQH5BPN2R2NT0L" device="" value="FNR5012S100MT 10uH"/>
 </parts>
 <sheets>
@@
 <attribute name="VALUE" x="590.296" y="260.096" size="1.27" layer="96"/>
 </instance>
-<instance part="LOW_BATT" gate="G$1" x="591.82" y="193.04" smashed="yes" rot="R270">
-<attribute name="NAME" x="596.265" y="194.31" size="1.27" layer="95" rot="R270" align="center"/>
-<attribute name="VALUE" x="589.026" y="194.31" size="1.27" layer="96" rot="R270" align="center"/>
+<instance part="LOW_BATT" gate="G$1" x="591.82" y="195.58" smashed="yes">
+<attribute name="NAME" x="594.36" y="194.818" size="1.778" layer="95" rot="R180" align="top-right"/>
+<attribute name="VALUE" x="594.36" y="192.278" size="1.778" layer="96" rot="R180" align="top-right"/>
 </instance>
 <instance part="R20" gate="G$1" x="591.82" y="203.2" smashed="yes" rot="R90">
@@
 <attribute name="VALUE" x="591.82" y="203.2" size="1.016" layer="96" font="vector" ratio="15" rot="R90" align="center"/>
 </instance>
-<instance part="LED2" gate="G$1" x="612.14" y="251.46" smashed="yes">
-<attribute name="NAME" x="610.87" y="255.905" size="1.27" layer="95" align="center"/>
-<attribute name="VALUE" x="610.87" y="248.666" size="1.27" layer="96" align="center"/>
+<instance part="LED2" gate="G$1" x="609.6" y="251.46" smashed="yes" rot="R90">
+<attribute name="NAME" x="610.362" y="254" size="1.778" layer="95" rot="R270" align="top-right"/>
+<attribute name="VALUE" x="612.902" y="254" size="1.778" layer="96" rot="R270" align="top-right"/>
 </instance>
 <instance part="R5" gate="G$1" x="599.44" y="251.46" smashed="yes">
@@
 <attribute name="VALUE" x="623.316" y="48.26" size="1.27" layer="96"/>
 </instance>
-<instance part="L2" gate="G$1" x="579.12" y="71.12" smashed="yes">
-<attribute name="NAME" x="568.96" y="76.2" size="1.778" layer="95"/>
-<attribute name="VALUE" x="568.96" y="66.04" size="1.778" layer="96" align="top-left"/>
-</instance>
 <instance part="U$85" gate="G$1" x="594.36" y="33.02" smashed="yes">
 <attribute name="VALUE" x="592.836" y="30.48" size="1.27" layer="96"/>
@@
 <attribute name="VALUE" x="551.18" y="-4.318" size="1.778" layer="96" rot="R180" align="center"/>
 </instance>
+<instance part="RPIBOOT3" gate="G$1" x="421.64" y="35.56" smashed="yes">
+<attribute name="NAME" x="419.1" y="38.1" size="1.778" layer="95" font="vector"/>
+<attribute name="VALUE" x="419.1" y="33.02" size="1.778" layer="96" font="vector"/>
+</instance>
+<instance part="L3" gate="G$1" x="579.12" y="71.12" smashed="yes">
+<attribute name="NAME" x="568.96" y="78.74" size="1.778" layer="95"/>
+<attribute name="VALUE" x="568.96" y="76.2" size="1.778" layer="96"/>
+</instance>
 </instances>
 <busses>
@@
 <wire x1="601.98" y1="71.12" x2="594.36" y2="71.12" width="0.1524" layer="91"/>
 <junction x="594.36" y="71.12"/>
-<pinref part="L2" gate="G$1" pin="2"/>
 <wire x1="594.36" y1="71.12" x2="591.82" y2="71.12" width="0.1524" layer="91"/>
+<pinref part="L3" gate="G$1" pin="2"/>
 </segment>
 </net>
@@
 </segment>
 <segment>
-<pinref part="L2" gate="G$1" pin="1"/>
 <wire x1="566.42" y1="71.12" x2="563.88" y2="71.12" width="0.1524" layer="91"/>
 <wire x1="563.88" y1="71.12" x2="563.88" y2="63.5" width="0.1524" layer="91"/>
 <pinref part="C17" gate="G$1" pin="1"/>
 <label x="563.88" y="71.12" size="1.778" layer="95" rot="R90" xref="yes"/>
+<pinref part="L3" gate="G$1" pin="1"/>
 </segment>
 </net>
@@
 <junction x="408.94" y="38.1"/>
 <label x="408.94" y="40.64" size="1.016" layer="95" rot="R90" xref="yes"/>
+<pinref part="RPIBOOT3" gate="G$1" pin="1"/>
+<wire x1="421.64" y1="35.56" x2="408.94" y2="35.56" width="0.1524" layer="91"/>
 </segment>
 </net>

Commit message: pcb
Parts:
- removed JOY_STICK, SOM_UART: BM04B-GHS-TBT(LF)(SN)(N), BM04B-GHS-TBT_LF__SN__N_:BM04B-GHS-TBT(LF)(SN)(N)
- removed JP6: S2B-PH-SM4-TB, SparkFun-Connectors:JST_2MM_MALE
- removed R29: 10K, Resistor:R-US_CHIP-0402(1005-METRIC)
- removed U8: MC74VHC1G14DFT1G, MC74VHC1G14DFT1G:MC74VHC1G14DFT1G
- added C28, C32, C33, C36: 10uF, Capacitor:C_CHIP-0402(1005-METRIC)
- added C31: 0.1uF, Capacitor:C_CHIP-0402(1005-METRIC)
- added C34, C35: 1uF, Capacitor:C_CHIP-0402(1005-METRIC)
- added GND36, GND37, GND40, GND41, GND42, GND7, RPIBOOT10, RPIBOOT11, RPIBOOT12, RPIBOOT6, RPIBOOT8, RPIBOOT9: DNP, SparkFun-Connectors:TEST-POINT3
- added H2, J3, J4, J5: BM04B-SRSS-TBCONN4_BM04B-SRSS_JST, 2024-05-18_10-24-10_Library:BM04B-SRSS-TBCONN4_BM04B-SRSS_JST
- added IC1: LIS3MDL, adafruit_sensor:LIS3MDL
- added Q4: NMOS_C7465427, Transistor:NMOSFETSOT23-GSD
- added RPIBOOT7: TEST-POINT3, SparkFun-Connectors:TEST-POINT3
- added U15: AP2112-3.3K, microbuilder:VREG_SOT23-5
- added U16: W25Q16JVUXIQ_TR, W25Q16JVUXIQ_TR:W25Q16JVUXIQ_TR
- added U17, U18, U19, U20, U21, U22, U23, U24: TPD1E1B04DPYRDPY2_TEX, 2024-05-19_00-17-33_Library:TPD1E1B04DPYRDPY2_TEX
- added U25: DRV2605LDGSR, DRV2605LDGSR:DRV2605LDGSR
- added U7: SN74LVC244ARWPRRWP0020A, 2024-05-18_09-46-26_Library:SN74LVC244ARWPRRWP0020A
- J1: value BM04B-GHS-TBT(LF)(SN)(N) -> SM03B-SRSS-TBCONN_SM03B-SRSS-TB_JST; device BM04B-GHS-TBT_LF__SN__N_:BM04B-GHS-TBT(LF)(SN)(N) -> 2024-05-21_05-27-43_Library:SM03B-SRSS-TBCONN_SM03B-SRSS-TB_JST
- R39: value 300k -> 10k
- U6: value W25Q128JVSIQSOIC_128JVSIQ_WIN-L -> LSM6DS3; device 2024-03-29_04-43-21_Library:W25Q128JVSIQSOIC_128JVSIQ_WIN-L -> adafruit_sensor:LSM6DS3
Connections:
- net SAM_EINK_ON renamed SAM_EINK_PWR
- removed net N$25: R29.1, SJ1.2
- removed net SAM_GPIO22: C2040.GPIO22
- removed net SAM_GPIO25: C2040.GPIO25
- new net 2A3: U7.2A3
- new net 2A4: U7.2A4
- new net 2Y3: U7.2Y3
- new net 2Y4: U7.2Y4
- new net HAP_3V3: C33.1, C35.1, U15.OUT, U25.EN, U25.VDD, U25.VDD/NC
- new net N$8: C31.1, IC1.C1
- new net SAM_BOOT: Q4.G, RPI-CM1G$1.GPIO16
- new net SAM_EINK_SWITCH: C2040.GPIO22, U7.1OE_N, U7.2OE_N
- new net SAM_GPIO23: C2040.GPIO23
- new net SOC_EINK_BUSY: RPI-CM1G$1.GPIO9, U7.1Y1
- new net SOC_EINK_CS: RPI-CM1G$1.GPIO8, U7.1A4
- new net SOC_EINK_D/C: RPI-CM1G$1.GPIO6, U7.1A3
- new net SOC_EINK_RESET: RPI-CM1G$1.GPIO13, U7.1A2
- new net SOC_SPI_CLK: RPI-CM1G$1.GPIO11, U7.2A1
- new net SOC_SPI_MOSI: RPI-CM1G$1.GPIO10, U7.2A2
- new net THERM: J1.2, SJ1.1
- new net U25_OUT+: H2.1, H2.2, U25.OUT+
- new net U25_OUT-: H2.3, H2.4, U25.OUT-
- net 3.3V: now also C28.1, C36.2, IC1.VDD, IC1.VDDIO, U6.VDD, U6.VDDIO; no longer C7.1, Q2.S, R43.1
- net 5.0V: now also J3.3; no longer J1.3
- net BATTERY_IN: now also J1.3; no longer JP6.+
- net EINK_BUSY: now also RPIBOOT9.1, U18.I/O, U7.1A1; no longer RPI-CM1G$1.GPIO9
- net EINK_CS: now also GND41.1, U20.I/O, U7.1Y4; no longer RPI-CM1G$1.GPIO8
- net EINK_D/C: now also RPIBOOT10.1, U19.I/O, U7.1Y3; no longer RPI-CM1G$1.GPIO6
- net EINK_RESET: now also GND40.1, U17.I/O, U7.1Y2; no longer RPI-CM1G$1.GPIO13
- net FAN_PWM: now also J3.1; no longer J1.1
- net GND: now also C28.2, C31.2, C32.2, C33.2, C34.1, C35.2, C36.1, IC1.GND, IC1.SDO, J1.1, J3.4, J4.4, J5.3, J5.4, Q4.S, U15.GND, U16.GND, U17.I/O_2, U18.I/O_2, U19.I/O_2, U20.I/O_2, U21.I/O_2, U22.I/O_2, U23.I/O_2, U24.I/O_2, U25.GND, U25.IN/TRIG, U6.SDO, U7.GND, U7.PAD; no longer J1.4, J1.SHIELD, JOY_STICK.4, JP6.-, SJ1.1, SOM_UART.4, U8.GND
- net N$16: now also C34.2, U25.REG; no longer Q3.G, U8.OUT_~Y
- net N$24: now also Q4.D
- net SAM_3V3: now also C7.1, J4.1, Q2.S, R43.1, U16.VCC, U7.VCC; no longer JOY_STICK.1, U6.VCC, U8.VCC
- net SAM_INTERUPT: now also RPIBOOT12.1
- net SAM_QSPI_SCLK: now also U16.CLK; no longer U6.CLK
- net SAM_QSPI_SCN: now also U16.!CS!; no longer U6./CS
- net SAM_QSPI_SD0: now also U16.IO0; no longer U6.DI_(IO0)
- net SAM_QSPI_SD1: now also U16.IO1; no longer U6.DO_(IO1)
- net SAM_QSPI_SD2: now also U16.IO2; no longer U6./WP_(IO2)
- net SAM_QSPI_SD3: now also U16.IO3; no longer U6./HOLD_OR_/RESET_(IO3)
- net SAM_SCL: now also C2040.GPIO25, J4.3, RPIBOOT8.1, U25.SCL; no longer C2040.GPIO23, JOY_STICK.3
- net SAM_SDA: now also GND37.1, J4.2, U25.SDA; no longer JOY_STICK.2
- net SCL1: now also IC1.SCL, RPIBOOT6.1, U6.SCL
- net SDA1: now also GND7.1, IC1.SDA, U6.SDA
- net SPI_CLK: now also RPIBOOT11.1, U21.I/O, U7.2Y1; no longer RPI-CM1G$1.GPIO11
- net SPI_MOSI: now also GND42.1, U22.I/O, U7.2Y2; no longer RPI-CM1G$1.GPIO10
- net SYS_PI_ON: now also Q3.G; no longer U8.IN_A
- net TACH: now also J3.2; no longer J1.2
- net TS: now also SJ1.2; no longer R29.2
- net TSCL: now also U23.I/O
- net TSDA: now also U24.I/O
- net UART_RXD0: now also J5.2; no longer SOM_UART.3
- net UART_RXD3_SAM: now also RPIBOOT7.1
- net UART_TXD0: now also J5.1; no longer SOM_UART.2
- net UART_TXD3_SAM: now also GND36.1
- net VOUT: now also C32.1, U15.EN, U15.IN
Other:
- note removed: "(COM-00906, COM-09940, COM-09119, COM-10613, ETC.)"
- note removed: "OPEN SOLDER JUMPER SJ1 AND ATTACH 10K POT TO JP4"
- note removed: "OPTIONAL EXTERNAL VOLUME CONTROL"
- moved on the sheet: BUD, BUP, BUS, GND34, Q3, R15, R16, R17, R18, R28, R33, R34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

Commit message: v0.7
Parts:
- removed J3: BM04B-SRSS-TBCONN4_BM04B-SRSS_JST, 2024-05-18_10-24-10_Library:BM04B-SRSS-TBCONN4_BM04B-SRSS_JST
- added J6: SM04B-SRSS-TBCONN_SM04B-SRSS-TB_JST, 2024-06-16_01-36-12_Library:SM04B-SRSS-TBCONN_SM04B-SRSS-TB_JST
Connections:
- net 5.0V: now also J6.3; no longer J3.3
- net FAN_PWM: now also J6.1; no longer J3.1
- net GND: now also J6.4; no longer J3.4
- net TACH: now also J6.2; no longer J3.2
Changed lines of the file:
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@@
 <part name="L3" library="LQH5BPN2R2NT0L" deviceset="LQH5BPN2R2NT0L" device="" value="FNR5012S100MT 10uH"/>
 <part name="U7" library="2024-05-18_09-46-26_Library" deviceset="SN74LVC244ARWPR" device="RWP0020A"/>
-<part name="J3" library="2024-05-18_10-24-10_Library" deviceset="BM04B-SRSS-TB" device="CONN4_BM04B-SRSS_JST"/>
 <part name="J4" library="2024-05-18_10-24-10_Library" deviceset="BM04B-SRSS-TB" device="CONN4_BM04B-SRSS_JST"/>
 <part name="J5" library="2024-05-18_10-24-10_Library" deviceset="BM04B-SRSS-TB" device="CONN4_BM04B-SRSS_JST"/>
@@
 <part name="U$111" library="microbuilder" deviceset="GND" device=""/>
 <part name="U$112" library="microbuilder" deviceset="GND" device=""/>
+<part name="J6" library="2024-06-16_01-36-12_Library" deviceset="SM04B-SRSS-TB" device="CONN_SM04B-SRSS-TB_JST"/>
 </parts>
 <sheets>
@@
 <attribute name="VALUE" x="632.1752" y="-36.6014" size="2.083" layer="96" ratio="6"/>
 </instance>
-<instance part="J3" gate="A" x="548.64" y="152.4" smashed="yes">
-<attribute name="NAME" x="552.8046" y="157.7086" size="2.083" layer="95" ratio="6"/>
-</instance>
 <instance part="J4" gate="A" x="937.26" y="241.3" smashed="yes">
 <attribute name="NAME" x="941.4246" y="246.6086" size="2.083" layer="95" ratio="6"/>
@@
 <attribute name="VALUE" x="-42.164" y="182.88" size="1.27" layer="96"/>
 </instance>
+<instance part="J6" gate="A" x="548.64" y="152.4" smashed="yes">
+<attribute name="NAME" x="552.8046" y="157.7086" size="2.083" layer="95" ratio="6"/>
+</instance>
 </instances>
 <busses>
@@
 <pinref part="C42" gate="G$1" pin="2"/>
 <wire x1="546.1" y1="139.7" x2="538.48" y2="139.7" width="0.1524" layer="91"/>
-<pinref part="J3" gate="A" pin="4"/>
+<pinref part="J6" gate="A" pin="4"/>
 </segment>
 <segment>
@@
 <wire x1="538.48" y1="147.32" x2="533.4" y2="147.32" width="0.1524" layer="91"/>
 <junction x="538.48" y="147.32"/>
-<pinref part="J3" gate="A" pin="3"/>
+<pinref part="J6" gate="A" pin="3"/>
 </segment>
 <segment>
@@
 <wire x1="546.1" y1="149.86" x2="546.1" y2="157.48" width="0.1524" layer="91"/>
 <junction x="546.1" y="149.86"/>
-<pinref part="J3" gate="A" pin="2"/>
+<pinref part="J6" gate="A" pin="2"/>
 </segment>
 </net>
@@
 <wire x1="548.64" y1="152.4" x2="535.94" y2="152.4" width="0.1524" layer="91"/>
 <label x="535.94" y="152.4" size="1.778" layer="95"/>
-<pinref part="J3" gate="A" pin="1"/>
+<pinref part="J6" gate="A" pin="1"/>
 </segment>
 </net>

Commit message: before modification, v0.7, for fateen and adam
Other:
- note added: "ACTIVE COOLING"
- note added: "AUDIO SUBSYSTEM"
- note added: "CAMERA"
- note added: "DIGITAL PERIPHERAL"
- note added: "EINK_SUBSYSTEM"
- note added: "HAPTIC MOTOR"
- note added: "MOTION SUBSYSTEM"
- note added: "PCIE M.2"
- note added: "POWER SUBSYSTEM"
- note added: "SAM"
- note added: "SOM"
- note added: "USB2.0"
- note removed: "CAMERA MODULE"
- note removed: "EINK HiGH VOLTAGE MODULE"
- moved on the sheet: BUD, BUP, BUS, C1, C10, C11, C12, C13, C14, C15, C16, C17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
