File: PCB/AI_EINK.sch (EAGLE design)
At the start: 206 parts, among them IC1 LIS3MDL, IC3 WM8960, J1 SM03B-SRSS-TBCONN_SM03B-SRSS-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, J2 C393939, J4 BM04B-SRSS-TBCONN4_BM04B-SRSS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, J5 BM04B-SRSS-TBCONN4_BM04B-SRSS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, J6 SM04B-SRSS-TBCONN_SM04B-SRSS-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, Q1 SI1308EDL-T1-GE3, Q2 DMG2307L, Q3 NMOS_C7465427, Q4 NMOS_C7465427, T1 MMUN2133LT1G, U1 TPS61092RSAR, U10 AP2112-3.3K, U11 AP2112-3.3K, U12 C233266, U13 TPD4EUSB30DQARDQA10, U14 OPA344, U15 AP2112-3.3K, U16 W25Q16JVUXIQ_TR, U17 TPD1E1B04DPYRDPY2_TEX, U18 TPD1E1B04DPYRDPY2_TEX, U19 TPD1E1B04DPYRDPY2_TEX, U2 MC74VHC1G14DFT1G, U20 TPD1E1B04DPYRDPY2_TEX, U21 TPD1E1B04DPYRDPY2_TEX, U22 TPD1E1B04DPYRDPY2_TEX, U23 TPD1E1B04DPYRDPY2_TEX, U24 TPD1E1B04DPYRDPY2_TEX, U25 DRV2605LDGSR, U3 BQ27441DRZR-G1A, U4 BQ24075, U5 MC74VHC1G14DFT1G OR C66196, U6 LSM6DS3, U7 SN74LVC244ARWPRRWP0020A, U9 EMC2301-1-ACZL-TRMSOP8_MC_MCH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, Y1 ABM8-272-T3

Commit message: ESP32
Parts:
- added C37, C38: 0.1uF, Capacitor:C_CHIP-0402(1005-METRIC)
- added C39, C54, C55: 10uF, Capacitor:C_CHIP-0402(1005-METRIC)
- added C52, C57: 220pF, Capacitor:C_CHIP-0402(1005-METRIC)
- added DISPLAY: C262642, 2024-03-29_02-21-27_Library:524372271CON_524372271_MOL
- added FB4, FB7: 120o, Filter:FBCHIP-0603(1608-METRIC)
- added J10, J11, J8, J9: SM04B-SRSS-TBCONN_SM04B-SRSS-TB_JST, 2024-06-16_01-36-12_Library:SM04B-SRSS-TBCONN_SM04B-SRSS-TB_JST
- added J3, J7: SM02B-SRSS-TB(LF)(SN), SM02B-SRSS-TB_LF__SN_:SM02B-SRSS-TB(LF)(SN)
- added R29: 8.2k, Resistor:R-US_CHIP-0402(1005-METRIC)
- added R46: 10K Trim, adafruit_electromech:R-TRIMM3314J
- added R48, R49: 30k, Resistor:R-US_CHIP-0402(1005-METRIC)
- added U$120, U$123: MOUNTINGHOLE2.5, microbuilder:MOUNTINGHOLE2.5
- added U8: PAM8302, microbuilder:AUDIOAMP_PAM8302A
Connections:
- net N$11 renamed PI_PWR_INDICATE
- removed net N$40: FB2.1, IC3.SPK_LP
- removed net N$41: FB3.1, IC3.SPK_LN
- removed net N$6: R20.2, T1.C
- new net IN+: R48.2, U8.IN_P
- new net IN-: R49.2, U8.IN_N
- new net LINPUT1: IC3.LINPUT1, J7.2
- new net LOW_BATT_P: J10.3, R20.2, T1.C
- new net N$25: C38.2, R49.1
- new net N$31: C37.2, R48.1
- new net N$32: C37.1, R29.2, R46.A
- new net OUT+: FB7.1, U8.VO_P
- new net OUT-: FB4.1, U8.VO_N
- new net SPK_LN: C38.1, FB3.1, IC3.SPK_LN, R46.E
- new net SPK_LP: FB2.1, IC3.SPK_LP, R29.1
- new net SPK_RN: IC3.SPK_RN
- new net SPK_RP: IC3.SPK_RP
- new net VO+: C57.1, FB7.2, J3.1
- new net VO-: C52.1, FB4.2, J3.2
- net !CHG!: now also J10.2
- net 3.3V: now also DISPLAY.22
- net 5.0V: now also C39.1, C54.1, C55.1, U8./SD, U8.VDD
- net BUTTON_D: now also J11.3
- net BUTTON_U: now also J11.2
- net DSI1_C_N: now also DISPLAY.8
- net DSI1_C_P: now also DISPLAY.9
- net DSI1_D0_N: now also DISPLAY.2
- net DSI1_D0_P: now also DISPLAY.3
- net DSI1_D1_N: now also DISPLAY.5
- net DSI1_D1_P: now also DISPLAY.6
- net DSI1_D2_N: now also DISPLAY.11
- net DSI1_D2_P: now also DISPLAY.12
- net DSI1_D3_N: now also DISPLAY.14
- net DSI1_D3_P: now also DISPLAY.15
- net GND: now also C39.2, C52.2, C54.2, C55.2, C57.2, DISPLAY.1, DISPLAY.10, DISPLAY.13, DISPLAY.16, DISPLAY.19, DISPLAY.4, DISPLAY.7, DISPLAY.P1, DISPLAY.P2, J10.4, J11.4, J7.1, J8.3, J8.4, J9.4, U8.GND
- net SAM_3V3: now also J11.1
- net SCL0: now also DISPLAY.20
- net SDA0: now also DISPLAY.21
- net USB_N: now also J9.3
- net USB_P: now also J9.2
- net VBUS: now also J8.1, J8.2, J9.1
- net VOUT: now also J10.1
Other:
- note added: "*TOP CONTACT"
- note added: "AUDIO AMP & External Mic"
- note added: "Adam"
- note added: "BUS BRK OUT"
- note added: "CAMERA MIPI 4 LANE"
- note added: "DISPLAY MIPI 4 LANE"
- note added: "Fateen"
- note added: "POWER INDICATOR BREAKOUT"
- note added: "ToDo: Ferrite (select w/high Z at high F, low Z at low F). Try to block everything >1MHz or so."
- note added: "WARNING: MEMS MIC WILL BE DAMAGED BY ISOPRO"
- note removed: "CAMERA"
- moved on the sheet: BUD, BUP, BUS, C27, C28, C29, C30, C31, C36, C45, C46, C47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
