File: PCB/AI_EINK.brd (EAGLE design)
At the start: 66 x 111.6 mm, 164 parts, among them IC3 WM8960, J1 BM04B-GHS-TBT(LF)(SN)(N), J3 524372471, Q1 SI1308EDL-T1-GE3, Q3 2A/20V/150mΩ, T1 MMUN2133LT1G, U1 TPS61090RSAR, U2 MC74VHC1G14DFT1G, U3 BQ27441DRZR-G1A, U4 BQ24075, U5 TLV74328, U6 TLV74315, U7 NE555DR, U8 SN74LV4040ARGYRRGY16_2P55X2P05, U9 EMC2301-1-ACZL-TRMSOP8_MC_MCH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

Commit message: a
Parts:
- removed BOOST_EN, COUNTER_CLR, GND10, GND11, GND29, PULSE_555: TEST-POINT3, SparkFun-Connectors:PAD.03X.03
- removed C40: 1nF, SparkFun-Capacitors:0603
- removed C41: 0.1uF, Capacitor:CAPC1608X85
- removed C51: 0.1uF, microbuilder:0603-NO
- removed C53, C55: 33pF, microbuilder:0603-NO
- removed C56: 10uF, microbuilder:0805-NO
- removed FB4: FERRITE, microbuilder:0805-NO
- removed FL1, FL2: BLM18HE152SN1D, BLM18HE152SN1D:BEADC1608X95N
- removed LEFTMIC, RIGHTMIC: (no value), microbuilder:SPW2430HR5H-B
- removed OV5647: DF30FC-24DP-0.4V(81), DF30FC-24DP-0.4V_81_:DF30FC-24DP
- removed Q3: 2A/20V/150mΩ, SparkFun-DiscreteSemi:SOT26
- removed R19: 10K, Resistor:RESC1608X60
- removed R21, R25, R26, R27: 10k, Resistor:RESC1608X60
- removed S2: FSMRA4JH04, FSMRA4JH04:FSMRA4JH04
- removed SJ5: (no value), SparkFun-Passives:PAD-JUMPER-3-2OF3_NC_BY_TRACE_YES_SILK_FULL_BOX
- removed SW1: (no value), adafruit:PUSHBUTTON_SMD_SJ
- removed U8: SN74LV4040ARGYRRGY16_2P55X2P05, 2024-03-07_02-24-03_Library:RGY16_2P55X2P05
- removed VR1: EC10E1220501, EC10E1220501:TRIM_EC10E1220501
- added B_D, B_S, B_U: FSMRA4JH04, FSMRA4JH04:FSMRA4JH04
- added C2040: RP2040TR13QFN56_7X7_RPI, 2024-03-10_01-36-20_Library:QFN56_7X7_RPI
- added C43, C44, C67, C69, C70, C71, C72, C73, C74, C77, C78, C81: 0.1uF, Capacitor:CAPC1608X85
- added C59, C60, C61, C62, C68, C79, C80: 10uF, Capacitor:CAPC1608X85
- added C75, C76: 1.0uF, Capacitor:CAPC1608X85
- added C82, C83: 15p, Capacitor:CAPC1608X85
- added D7: PMIC, SparkFun-LED:LED-0603
- added FB2, FB5: Ferrite, microbuilder:0805
- added FL3, FL4, FL5: BLM18HE152SN1D, BLM18HE152SN1D:BEADC1608X95N
- added GND34, USB_BOOT_N: TEST-POINT3, SparkFun-Connectors:PAD.03X.03
- added Q2: 2.5A/30V, User-Submitted:SOT23-3
- added R31, R32: 27, resistor:R0603
- added R34, R35: 1k, resistor:R0603
- added R36, R37: 200K, resistor:R0603
- added SJ2, SJ3: (no value), SparkFun-Passives:PAD-JUMPER-3-2OF3_NC_BY_TRACE_YES_SILK_FULL_BOX
- added SPI_FLASH_SAM: W25Q128JVBIQTFBGA_128JVBIQ_WIN, 2024-03-10_02-04-46_Library:TFBGA_128JVBIQ_WIN
- added U10, U11: AP2112-3.3K, microbuilder:SOT23-5
- added U12: SPU0410LR5H-QB, SPU0410LR5H-QB:XDCR_SPU0410LR5H-QB
- added Y1: ABM8-272-T3, ABM8-272-T3:ABM8272T3
- C1, C2, C24, C26, C3, C31, C32, C33, C34, C35, C45, C46, C57, C65, C66, C7: device microbuilder:0805-NO -> Capacitor:CAPC1608X85
- C16, C17, C18, C4, C42: device microbuilder:0805_10MGAP -> Capacitor:CAPC1608X85
- C19, C20: device SparkFun-Capacitors:0603-CAP -> Capacitor:CAPC1608X85
- C21, C23: device SparkFun-Capacitors:0805-CAP -> Capacitor:CAPC1608X85
- C22: device SparkFun-Capacitors:1206-CAP -> Capacitor:CAPC1608X85
- C25: value 0.1uF -> 1.0uF; device microbuilder:0603-NO -> Capacitor:CAPC1608X85
- C27, C30, C47, C48, C49, C50, C52, C54, C58, C63, C64: device microbuilder:0603-NO -> Capacitor:CAPC1608X85
- C28: value 1uF -> 10uF
- C29: value 0.1uF -> 10uF
- C36, C37, C38, C39: value 1nF -> 10uF; device SparkFun-Capacitors:0603 -> Capacitor:CAPC1608X85
- J2: value (none) -> C393939
- R1, R2: device microbuilder:_0805MP -> resistor:R0603
- R10, R8: device rcl:R0603 -> resistor:R0603
- R11, R17, R30, R9: device Resistor:RESC1608X60 -> resistor:R0603
- R13, R20, R3, R4, R5: device microbuilder:0805-NO -> resistor:R0603
- R14: value 10K -> 1K; device microbuilder:0603-NO -> resistor:R0603
- R15, R18, R22, R23, R24, R29, R33: device SparkFun-Resistors:0603-RES -> resistor:R0603
- R16: value 280k -> 10k; device Resistor:RESC1608X60 -> resistor:R0603
- R28: value 1k -> 10k; device rcl:R0603 -> resistor:R0603
- R6, R7: device SparkFun-Passives:0603-RES -> resistor:R0603
- U7: value NE555DR -> TLV74318PDBVRDBV0005A_L; device IC:SOIC-8N -> 2024-03-10_03-34-55_Library:DBV0005A_L
- moved OV5674 281.8 mm to (43.2, 95.8), turned to 270 degrees
- moved C42 211.6 mm to (36.2, 37.4), turned to 90 degrees
- moved J1 203.1 mm to (41.7, 38.8)
- moved R30 197.5 mm to (41.8, 26.1), turned to 270 degrees
- moved R17 184.5 mm to (59.0, 87.5), turned to 270 degrees
- moved U9 180.0 mm to (38.5, 31.9), turned to 270 degrees
- moved C29 154.6 mm to (38.3, 91.4), turned to 270 degrees
- moved C28 146.7 mm to (34.8, 91.4), turned to 270 degrees
- moved R16 129.0 mm to (9.36, 54.3), turned to 90 degrees
- moved U7 125.9 mm to (32.0, 91.4)
- moved R18 66.6 mm to (40.7, 103.3), turned to 180 degrees
- moved R15 63.8 mm to (44.6, 103.3)
- moved R14 58.3 mm to (21.3, 33.7), turned to 0 degrees
- moved RPIBOOT3 47.7 mm to (40.8, 85.4)
- moved GND25 45.9 mm to (42.7, 85.4)
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Connections:
- removed net !PGOOD!: SJ5.1, U4.7
- removed net BUTTON: RPI-CM1.24, S2.2
- removed net COUNTER_CLR: COUNTER_CLR.P$1, Q3.D2, R19.2, U8.11, U8.2
- removed net LINPUT1: C56.2, IC3.4
- removed net N$20: R21.2, R26.1, VR1.A
- removed net N$22: R25.2, R27.1, VR1.B
- removed net N$28: R23.2, SJ5.2
- removed net N$31: C53.1, FB4.1, LEFTMIC.1
- removed net N$37: C55.1, C56.1, FB4.2
- removed net POWER_OFF_MCU: Q3.G2, RPI-CM1.41
- removed net POWER_SWITCH_N: Q3.G1, R17.2, RPI-CM1.37, SW1.P$2
- removed net PULSE_555: PULSE_555.P$1, U7.3, U8.10
- removed net PWM_FAN: RPI-CM1.55
- removed net ROT1: C41.1, R25.1, RPI-CM1.46
- removed net ROT2: C29.1, R21.1, RPI-CM1.50
- removed net TRIG: C28.1, R16.1, U7.2, U7.6
- removed net V_OUT: Q3.S1, Q3.S2, S1.1, SW1.P$1, U8.16
- new net AF_EN: OV5674.18
- new net BUTTON_D: B_D.2, C2040.29
- new net BUTTON_S: B_S.2, C2040.27
- new net BUTTON_U: B_U.2, C2040.28
- new net N$24: R34.2, USB_BOOT_N.P$1
- new net N$26: C83.2, R35.2, Y1.3
- new net N$27: R37.1, S1.3
- new net OUT: C62.1, C69.1, FB2.2, U10.5
- new net PI_1V8: RPI-CM1.88, RPI-CM1.90
- new net PWDN: OV5674.19, SJ3.2
- new net RESET: OV5674.22, SJ2.2
- new net SAM_1V1: C2040.23, C2040.45, C2040.50, C76.1, C77.1, C78.1
- new net SAM_3V3: B_D.1, B_S.1, B_U.1, C2040.1, C2040.10, C2040.22, C2040.33, C2040.42, C2040.43, C2040.44, C2040.48, C2040.49, C43.1, C44.1, C70.1, C71.1, C72.1, C73.1, C74.1, C75.1, C80.1, C81.1, D7.A, R16.2, R17.2, R28.2, SPI_FLASH_SAM.B4, U11.5
- new net SAM_GPIO0: C2040.2
- new net SAM_GPIO1: C2040.3
- new net SAM_GPIO10: C2040.13
- new net SAM_GPIO11: C2040.14
- new net SAM_GPIO12: C2040.15
- new net SAM_GPIO13: C2040.16
- new net SAM_GPIO14: C2040.17
- new net SAM_GPIO15: C2040.18
- new net SAM_GPIO2: C2040.4
- new net SAM_GPIO22: C2040.34
- new net SAM_GPIO23: C2040.35
- new net SAM_GPIO24: C2040.36
- new net SAM_GPIO25: C2040.37
- new net SAM_GPIO26/ADC0: C2040.38
- new net SAM_GPIO27/ADC1: C2040.39
- new net SAM_GPIO28/ADC2: C2040.40
- new net SAM_GPIO29/ADC3: C2040.41
- new net SAM_GPIO3: C2040.5
- new net SAM_GPIO4: C2040.6
- new net SAM_GPIO5: C2040.7
- new net SAM_GPIO6: C2040.8
- new net SAM_GPIO7: C2040.9
- new net SAM_GPIO8: C2040.11
- new net SAM_GPIO9: C2040.12
- new net SAM_QSPI_SCLK: C2040.52, SPI_FLASH_SAM.B2
- new net SAM_QSPI_SCN: C2040.56, R34.1, SPI_FLASH_SAM.C2
- new net SAM_QSPI_SD0: C2040.53, SPI_FLASH_SAM.D3
- new net SAM_QSPI_SD1: C2040.55, SPI_FLASH_SAM.D2
- new net SAM_QSPI_SD2: C2040.54, SPI_FLASH_SAM.C4
- new net SAM_QSPI_SD3: C2040.51, SPI_FLASH_SAM.D4
- new net SAM_RUN: C2040.26
- new net SAM_SWCLK: C2040.24
- new net SAM_SWD: C2040.25
- new net SAM_USB_DM: C2040.46, R32.2
- new net SAM_USB_DP: C2040.47, R31.2
- new net SAM_XIN: C2040.20, C82.1, Y1.1
- new net SAM_XOUT: C2040.21, R35.1
- new net STROBE: OV5674.20
- new net SYS_POW_SAM: C2040.32, Q2.1
- net 1.5V: now also FL3.1; no longer FL2.1
- net 1.8V: now also C25.1, C28.1, C29.1, FL4.1, SJ2.3, SJ3.1, U7.5; no longer RPI-CM1.88, RPI-CM1.90
- net 2.8V: now also FL5.1; no longer C38.1, FL1.1, OV5647.P$19
- net 3.3V: now also C36.1, C37.1, C38.1, C39.1, U7.1, U7.3; no longer C25.1, R26.2, R27.2, R28.2, S2.1
- net 5.0V: now also C59.1, C60.1, C61.1, U10.1, U10.3
- net AGND: now also C67.2, C68.2, FB5.1
- net AVDD: now also C67.1, C68.1, FB2.1, U12.4; no longer C51.1, LEFTMIC.4, RIGHTMIC.4
- net BOOST_EN: now also Q2.3, R36.1; no longer BOOST_EN.P$1, U8.5
- net CAM0_C_N: now also OV5674.8; no longer OV5647.P$8
- net CAM0_C_P: now also OV5674.9; no longer OV5647.P$7
- net CAM0_D0_N: now also OV5674.2; no longer OV5647.P$10
- net CAM0_D0_P: now also OV5674.3; no longer OV5647.P$9
- net CAM0_D1_N: now also OV5674.5; no longer OV5647.P$6
- net CAM0_D1_P: now also OV5674.6; no longer OV5647.P$5
- net EINK_BUSY: now also RPI-CM1.34; no longer RPI-CM1.26
- net GND: now also C2040.19, C2040.57, C43.2, C44.2, C59.2, C60.2, C61.2, C62.2, C69.2, C70.2, C71.2, C72.2, C73.2, C74.2, C75.2, C76.2, C77.2, C78.2, C79.2, C80.2, C81.2, C82.2, C83.1, FB5.2, GND34.P$1, OV5674.1, OV5674.10, OV5674.12, OV5674.21, OV5674.4, OV5674.7, R16.1, R23.2, R36.2, R37.2, SJ2.1, SJ3.3, SPI_FLASH_SAM.B3, U10.2, U11.2, U12.2, U12.3, U12.5, U12.6, U7.2, Y1.2, Y1.4; no longer C40.2, C41.2, C51.2, C53.2, C55.2, GND10.P$1, GND11.P$1, GND29.P$1, LEFTMIC.2, LEFTMIC.3, OV5647.P$13, OV5647.P$15, OV5647.P$17, R19.1, RIGHTMIC.2, RIGHTMIC.3, S1.3, SJ5.3, U7.1, U8.8, VR1.C
- net I2S_BCLK: now also RPI-CM1.49; no longer RPI-CM1.25
- net I2S_DIN: now also RPI-CM1.27; no longer RPI-CM1.31
- net I2S_DOUT: now also RPI-CM1.25; no longer RPI-CM1.29
- net I2S_LRCLK: now also RPI-CM1.26; no longer RPI-CM1.27
- net N$10: now also FL4.2, OV5674.15; no longer OV5647.P$24, R14.1
- net N$13: now also FL3.2, OV5674.13, OV5674.14; no longer C39.1, C40.1, FL2.2, OV5647.P$20
- net N$18: now also D7.C, R14.1; no longer Q3.D1, R16.2, U7.4, U7.7, U7.8
- net N$29: now also U12.1; no longer RIGHTMIC.1
- net N$8: now also FL5.2, OV5674.16, OV5674.17; no longer C36.1, C37.1, FL1.2, OV5647.P$18
- net RFC_MCLK: now also OV5674.11; no longer OV5647.P$14
- net SCL: now also OV5674.23; no longer OV5647.P$11
- net SDA: now also OV5674.24; no longer OV5647.P$12
- net USB_N: now also R32.1
- net USB_P: now also R31.1
- net VOUT: now also C79.1, Q2.2, S1.1, U11.1, U11.3
Routing:
- net SAM_3V3: track 0.00 -> 193.2 mm, vias 0 -> 7
- net BUTTON_S: track 0.00 -> 90.1 mm, vias 0 -> 6
- net LINPUT1: track 88.8 -> 0.00 mm, vias 2 -> 0
- net VOUT: track 14.2 -> 91.1 mm, vias 4 -> 11
- net BUTTON_U: track 0.00 -> 64.5 mm, vias 0 -> 2
- net BUTTON_D: track 0.00 -> 58.6 mm, vias 0 -> 4
- net AVDD: track 135.3 -> 86.2 mm, vias 11 -> 4
- net SAM_1V1: track 0.00 -> 38.4 mm, vias 0 -> 4
- net SCL: track 160.0 -> 197.5 mm, vias 9 -> 13
- net 3.3V: track 345.3 -> 308.1 mm
- net SYS_POW_SAM: track 0.00 -> 36.8 mm, vias 0 -> 2
- net BUTTON: track 36.1 -> 0.00 mm, vias 1 -> 0
- net ROT1: track 36.0 -> 0.00 mm, vias 2 -> 0
- net SDA: track 163.5 -> 199.1 mm, vias 11 -> 15
- net CAM0_D0_N: track 15.4 -> 46.0 mm, vias 2 -> 4
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Other:
- outline, holes or cut-outs redrawn

Commit message: a
Parts:
- removed B_D, B_S, B_U: FSMRA4JH04, FSMRA4JH04:FSMRA4JH04
- removed Q2: 2.5A/30V, User-Submitted:SOT23-3
- removed RF1: ST25DVXX_TSSOP, microbuilder:TSSOP8-4.4MM
- added BUD, BUP, BUS: EVQ-P7A01P, EVQ-P7A01P:SW_EVQ-P7A01P
- added Q3: NMOS_C7465427, Transistor:SOT23
- added U8: ST25DV64K-IER6S3SOIC_IER6S3_STM, 2024-03-10_23-40-44_Library:SOIC_IER6S3_STM
- GND, GND13, GND22, GND25, GND26, GND27, GND34, RPIBOOT, RPIBOOT1, RPIBOOT2, RPIBOOT3, RPIBOOT4, USB_BOOT_N: value TEST-POINT3 -> DNP
- JP6: value (none) -> S2B-PH-SM4-TB
- S1: value (none) -> C963206
- SJ1, SJ2, SJ3, SJ6: value (none) -> DNP
- moved C54 7.48 mm to (3.67, 77.8)
- moved C57 7.48 mm to (3.67, 79.7)
- moved R6 6.35 mm to (54.3, 14.5)
- moved C16 0.15 mm to (32.8, 16.5), turned to 270 degrees
Connections:
- net 3.3V: now also U8.8; no longer RF1.8
- net BOOST_EN: now also Q3.3, R36.2; no longer Q2.3, R36.1
- net BUTTON_D: now also BUD.2_1, BUD.2_2; no longer B_D.2
- net BUTTON_S: now also BUS.2_1, BUS.2_2; no longer B_S.2
- net BUTTON_U: now also BUP.2_1, BUP.2_2; no longer B_U.2
- net GND: now also Q3.2, U8.4; no longer R36.2, RF1.4
- net GPO: now also U8.7; no longer RF1.7
- net N$16: now also U8.2; no longer RF1.2
- net N$32: now also U8.3; no longer RF1.3
- net SAM_3V3: now also BUD.1_1, BUD.1_2, BUP.1_1, BUP.1_2, BUS.1_1, BUS.1_2; no longer B_D.1, B_S.1, B_U.1
- net SCL: now also U8.6; no longer RF1.6
- net SDA: now also U8.5; no longer RF1.5
- net SYS_POW_SAM: now also Q3.1; no longer Q2.1
- net VEH: now also U8.1; no longer RF1.1
- net VOUT: now also R36.1; no longer Q2.2
Routing:
- net BUTTON_S: track 90.1 -> 100.3 mm
- net N$36: track 3.88 -> 11.4 mm
- net RINPUT1: track 66.7 -> 59.4 mm
- net SAM_3V3: track 193.2 -> 200.3 mm, vias 7 -> 8
- net ISET: track 4.77 -> 11.5 mm
- net BUTTON_D: track 58.6 -> 65.2 mm, vias 4 -> 8
- net BOOST_EN: track 5.98 -> 11.3 mm
- net USB_N: track 81.8 -> 86.6 mm, vias 2 -> 4
- net BUTTON_U: track 64.5 -> 68.8 mm
- net GND: track 32.1 -> 28.1 mm, vias 203 -> 252
- net USB_P: track 84.4 -> 87.2 mm, vias 2 -> 4
- net SDA: track 199.1 -> 201.4 mm
- net SCL: track 197.5 -> 199.3 mm
- net VOUT: track 91.1 -> 89.6 mm
- net SYS_POW_SAM: track 36.8 -> 38.2 mm
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
Commit message: PCB
Parts:
- added C40, C41, C51, C53: 10uF, Capacitor:CAPC1608X85
- C22: value 1.0uF -> 10uF
- moved C22 72.9 mm to (-3.81, -23.1), turned to 0 degrees
Connections:
- net GND: now also C40.2, C41.2, C51.2, C53.2
- net VBUS: now also C53.1
- net V_BATT: now also C40.1, C41.1, C51.1

Commit message: pcb before downsize
Parts:
- U1: value TPS61090RSAR -> TPS61092RSAR
Connections:
- new net N$20: RPI-CM1.29
- new net N$22: RPI-CM1.41
- new net N$28: RPI-CM1.55
Changed lines of the file:
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@@
 <attribute name="BOM" value="EXCLUDE" x="97.012" y="12.001" size="1.778" layer="27" display="off"/>
 </element>
-<element name="U1" library="microbuilder" package="PVQFN-16" value="TPS61090RSAR" x="53.434" y="35.658" smashed="yes">
+<element name="U1" library="microbuilder" package="PVQFN-16" value="TPS61092RSAR" x="53.434" y="35.658" smashed="yes">
 <attribute name="NAME" x="51.41" y="38.54" size="0.4064" layer="25" ratio="18"/>
 <attribute name="VALUE" x="51.31" y="32.418" size="0.4064" layer="27" ratio="10"/>
@@
 <contactref element="U8" pad="7"/>
 </signal>
+<signal name="N$20">
+<contactref element="RPI-CM1" pad="29"/>
+</signal>
+<signal name="N$22">
+<contactref element="RPI-CM1" pad="41"/>
+</signal>
+<signal name="N$28">
+<contactref element="RPI-CM1" pad="55"/>
+</signal>
 </signals>

Commit message: kevin commit
Parts:
- removed R37: 200K, resistor:R0603
- removed S1: C963206, SparkFun-Electromechanical:SWITCH-SPST-SMD-A
Connections:
- removed net N$27: R37.1, S1.3
- net BOOST_EN: no longer S1.2
- net GND: no longer R37.2
- net VOUT: no longer S1.1
Routing:
- net BOOST_EN: track 11.3 -> 8.99 mm
- net N$27: track 2.16 -> 0.00 mm

Commit message: PCB V3
Parts:
- removed ANT1: NFC_ANTENNA_25X15, microbuilder:NFCANT_25X15
- removed C25, C30: 1.0uF, Capacitor:CAPC1608X85
- removed C27, C70, C78, C81: 0.1uF, Capacitor:CAPC1608X85
- removed C28, C29, C31, C32, C33, C34, C35, C36, C37, C38, C39, C41, C51: 10uF, Capacitor:CAPC1608X85
- removed FB10, FB9: 120o, microbuilder:0805-NO
- removed FL3, FL4, FL5: BLM18HE152SN1D, BLM18HE152SN1D:BEADC1608X95N
- removed GND25, RPIBOOT3: DNP, SparkFun-Connectors:PAD.03X.03
- removed J3: 524372471, 2024-02-19_09-48-43_Library:CON_524372471_MOL
- removed OSC1: 24MHz 3.3V Oscillator, microbuilder:OSC_3.2X2.5MM
- removed OV5674: DF30FC-24DS-0.4V(82)CONN_DF30FC-24DS-0.4V(82)_HIR, 2024-03-07_05-07-01_Library:CONN_DF30FC-24DS-0.4V(82)_HIR
- removed SJ2, SJ3: DNP, SparkFun-Passives:PAD-JUMPER-3-2OF3_NC_BY_TRACE_YES_SILK_FULL_BOX
- removed SPI_FLASH_SAM: W25Q128JVBIQTFBGA_128JVBIQ_WIN, 2024-03-10_02-04-46_Library:TFBGA_128JVBIQ_WIN
- removed U$10, U$11, U$94, U$95: MOUNTINGHOLE2.5, microbuilder:MOUNTINGHOLE_2.5_PLATED
- removed U7: TLV74318PDBVRDBV0005A_L, 2024-03-10_03-34-55_Library:DBV0005A_L
- added CAMERA: 524372271CON_524372271_MOL, 2024-03-29_02-21-27_Library:CON_524372271_MOL
- added EINK_524352471: 524372471, 2024-02-19_09-48-43_Library:CON_524372471_MOL
- added FB1, FB4: FERRITE_BEAD, Filter:BEADC1608X95N
- added JOY_STICK: BM04B-GHS-TBT(LF)(SN)(N), BM04B-GHS-TBT_LF__SN__N_:JST_BM04B-GHS-TBT(LF)(SN)(N)
- added M.2KEYM(NGFF): 1-2199119-5, 1-2199119-5:TE_1-2199119-5
- added Q2: NMOS_C7465427, Transistor:SOT23
- added R19: 5.1K, Resistor:RESC1005X40
- added R21: 5.1k, Resistor:RESC1005X40
- added R25, R26: 4.7K, Resistor:RESC1005X40
- added U13: TPD4EUSB30DQARDQA10, 2024-03-29_01-35-38_Library:DQA10
- C1, C10, C11, C12, C13, C14, C15, C16, C17, C19, C2, C20, C21, C22, C23, C26, C3, C4, C40, C43, C44, C45, C46, C47, C48, C49, C5, C50, C52, C53, C54, C57, C58, C59, C60, C61, C62, C63, C64, C65, C66, C67, C68, C69, C7, C71, C72, C73, C74, C75, C76, C77, C79, C8, C80, C82, C83, C9: device Capacitor:CAPC1608X85 -> Capacitor:CAPC1005X60
- C24: value 10uF -> 0.1uF; device Capacitor:CAPC1608X85 -> Capacitor:CAPC1005X60
- FB2, FB5: value Ferrite -> FERRITE_BEAD; device microbuilder:0805 -> Filter:BEADC1608X95N
- FB3: value Ferrite -> FERRITE_BEAD; device microbuilder:0805-NO -> Filter:BEADC1608X95N
- R1, R10, R11, R13, R14, R15, R16, R17, R18, R2, R20, R22, R23, R24, R28, R29, R3, R30, R31, R32, R33, R34, R35, R36, R4, R5, R6, R7, R8, R9: device resistor:R0603 -> Resistor:RESC1005X40
- U5: value TLV74328 -> MC74VHC1G14DFT1G; device adafruit_power:SOT23-5 -> MC74VHC1G14DFT1G:SOT65P210X110-5N
- U6: value TLV74315 -> W25Q128JVSIQSOIC_128JVSIQ_WIN-L; device adafruit_power:SOT23-5 -> 2024-03-29_04-43-21_Library:SOIC_128JVSIQ_WIN-L
- U8: value ST25DV64K-IER6S3SOIC_IER6S3_STM -> MC74VHC1G14DFT1G; device 2024-03-10_23-40-44_Library:SOIC_IER6S3_STM -> MC74VHC1G14DFT1G:SOT65P210X110-5N
- moved U8 87.8 mm to (53.3, 9.02), turned to 90 degrees
- moved FB3 82.3 mm to (52.6, 22.6)
- moved U5 80.6 mm to (17.8, 20.1)
- moved C7 80.3 mm to (19.9, 18.5), turned to 90 degrees
- moved RPIBOOT2 71.3 mm to (58.0, 88.8)
- moved C53 68.6 mm to (38.0, 24.6), turned to 90 degrees
- moved C26 67.1 mm to (37.6, 28.3), turned to 90 degrees
- moved GND13 65.9 mm to (58.0, 87.4)
- moved C22 64.5 mm to (39.5, 24.6), turned to 90 degrees
- moved GND 56.9 mm to (14.8, 7.05)
- moved C24 56.4 mm to (22.5, 44.2)
- moved C40 56.0 mm to (45.7, 22.9)
- moved U6 55.4 mm to (17.3, 42.3), turned to 0 degrees
- moved R15 51.7 mm to (36.7, 52.2), turned to 90 degrees
- moved R18 51.4 mm to (35.3, 52.2), turned to 90 degrees
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Connections:
- removed net 1.5V: C30.1, C34.1, C35.1, FL3.1, U6.5
- removed net 1.8V: C25.1, C28.1, C29.1, FL4.1, RPIBOOT3.P$1, SJ2.3, SJ3.1, U7.5
- removed net 2.8V: C24.1, C31.1, FL5.1, U5.5
- removed net AF_EN: OV5674.18
- removed net GPO: U8.7
- removed net N$10: FL4.2, OV5674.15
- removed net N$13: FL3.2, OV5674.13, OV5674.14
- removed net N$20: RPI-CM1.29
- removed net N$22: RPI-CM1.41
- removed net N$28: RPI-CM1.55
- removed net N$32: ANT1.P$1, U8.3
- removed net PWDN: OV5674.19, SJ3.2
- removed net RESET: OV5674.22, SJ2.2
- removed net RFC_MCLK: OSC1.3, OV5674.11
- removed net SAM_GPIO0: C2040.2
- removed net SAM_GPIO10: C2040.13
- removed net SAM_GPIO11: C2040.14
- removed net SAM_GPIO12: C2040.15
- removed net SAM_GPIO13: C2040.16
- removed net SAM_GPIO14: C2040.17
- removed net SAM_GPIO15: C2040.18
- removed net SAM_GPIO23: C2040.35
- removed net SAM_GPIO24: C2040.36
- removed net SAM_GPIO9: C2040.12
- removed net SCL: IC3.17, OV5674.23, R18.1, RPI-CM1.56, U3.2, U8.6, U9.2
- removed net SDA: IC3.18, OV5674.24, R15.1, RPI-CM1.58, U3.1, U8.5, U9.1
- removed net STROBE: OV5674.20
- removed net SYS_POW_SAM: C2040.32, Q3.1
- removed net VEH: U8.1
- new net 3V3_EINK: C17.1, C9.1, EINK_524352471.10, EINK_524352471.9, L2.1, Q2.2
- new net CAM1_C_N: CAMERA.8, RPI-CM1.127
- new net CAM1_C_P: CAMERA.9, RPI-CM1.129
- new net CAM1_D0_N: CAMERA.2, RPI-CM1.115
- new net CAM1_D0_P: CAMERA.3, RPI-CM1.117
- new net CAM1_D1_N: CAMERA.5, RPI-CM1.121
- new net CAM1_D1_P: CAMERA.6, RPI-CM1.123
- new net CAM1_D2_N: CAMERA.11, RPI-CM1.133
- new net CAM1_D2_P: CAMERA.12, RPI-CM1.135
- new net CAM1_D3_N: CAMERA.14, RPI-CM1.139
- new net CAM1_D3_P: CAMERA.15, RPI-CM1.141
- new net DSI0_C_N: RPI-CM1.169
- new net DSI0_C_P: RPI-CM1.171
- new net DSI0_D0_N: RPI-CM1.157
- new net DSI0_D0_P: RPI-CM1.159
- new net DSI0_D1_N: RPI-CM1.163
- new net DSI0_D1_P: RPI-CM1.165
- new net DSI1_C_N: RPI-CM1.187
- new net DSI1_C_P: RPI-CM1.189
- new net DSI1_D0_N: RPI-CM1.175
- new net DSI1_D0_P: RPI-CM1.177
- new net DSI1_D1_N: RPI-CM1.181
- new net DSI1_D1_P: RPI-CM1.183
- new net DSI1_D2_N: RPI-CM1.193
- new net DSI1_D2_P: RPI-CM1.195
- new net DSI1_D3_N: RPI-CM1.194
- new net DSI1_D3_P: RPI-CM1.196
- new net EXT_VCC_PCIE: M.2KEYM(NGFF).12, M.2KEYM(NGFF).14, M.2KEYM(NGFF).16, M.2KEYM(NGFF).18, M.2KEYM(NGFF).2, M.2KEYM(NGFF).4, M.2KEYM(NGFF).70, M.2KEYM(NGFF).72, M.2KEYM(NGFF).74
- new net GND_2: U13.3
- new net HDMI0_CEC: RPI-CM1.151
- new net HDMI0_CLK_N: RPI-CM1.190
- new net HDMI0_CLK_P: RPI-CM1.188
- new net HDMI0_HOTPLUG: RPI-CM1.153
- new net HDMI0_SCL: RPI-CM1.200
- new net HDMI0_SDA: RPI-CM1.199
- new net HDMI0_TX0_N: RPI-CM1.184
- new net HDMI0_TX0_P: RPI-CM1.182
- new net HDMI0_TX1_N: RPI-CM1.178
- new net HDMI0_TX1_P: RPI-CM1.176
- new net HDMI0_TX2_N: RPI-CM1.172
- new net HDMI0_TX2_P: RPI-CM1.170
- new net HDMI1_CEC: RPI-CM1.149
- new net HDMI1_CLK_N: RPI-CM1.166
- new net HDMI1_CLK_P: RPI-CM1.164
- new net HDMI1_HOTPLUG: RPI-CM1.143
- new net HDMI1_SCL: RPI-CM1.147
- new net HDMI1_SDA: RPI-CM1.145
- new net HDMI1_TX0_N: RPI-CM1.160
- new net HDMI1_TX0_P: RPI-CM1.158
- new net HDMI1_TX1_N: RPI-CM1.154
- new net HDMI1_TX1_P: RPI-CM1.152
- new net HDMI1_TX2_N: RPI-CM1.148
- new net HDMI1_TX2_P: RPI-CM1.146
- new net N$27: J2.B5, R21.2
- new net N$30: J2.A5, R19.2
- new net PCIE_!RST: M.2KEYM(NGFF).50, RPI-CM1.109
- new net PCIE_CLK_!REQ: M.2KEYM(NGFF).52, RPI-CM1.102
- new net PCIE_CLK_N: M.2KEYM(NGFF).53, RPI-CM1.112
- new net PCIE_CLK_P: M.2KEYM(NGFF).55, RPI-CM1.110
- new net PCIE_RX_N: M.2KEYM(NGFF).41, RPI-CM1.118
- new net PCIE_RX_P: M.2KEYM(NGFF).43, RPI-CM1.116
- new net PCIE_TX_N: M.2KEYM(NGFF).47, RPI-CM1.124
- new net PCIE_TX_P: M.2KEYM(NGFF).49, RPI-CM1.122
- new net RESERVED@104: RPI-CM1.104
- new net RESERVED@106: RPI-CM1.106
- new net SAM_EINK_ON: C2040.12, U5.2
- new net SAM_INTERUPT: C2040.2, RPI-CM1.46
- new net SAM_SCL: C2040.35, JOY_STICK.3, R26.1, U3.2
- new net SAM_SDA: C2040.36, JOY_STICK.2, R25.1, U3.1
- new net SCL0: CAMERA.20, RPI-CM1.80
- new net SCL1: IC3.17, R18.1, RPI-CM1.56, U9.2
- new net SDA0: CAMERA.21, RPI-CM1.82
- new net SDA1: IC3.18, R15.1, RPI-CM1.58, U9.1
- new net SYS_PI_ON: C2040.32, U8.2
- new net USB_OTG_ID: RPI-CM1.101
- new net VDAC_COMP: RPI-CM1.111
- net 3.3V: now also CAMERA.22, Q2.3; no longer C17.1, C26.1, C27.1, C32.1, C33.1, C36.1, C37.1, C38.1, C39.1, C9.1, J3.10, J3.9, L2.1, OSC1.1, OSC1.4, U5.1, U5.3, U6.1, U6.3, U7.1, U7.3, U8.8
- net AGND: now also FB5.2; no longer FB5.1
- net AVDD: now also FB1.2; no longer FB2.1
- net CAM0_C_N: no longer OV5674.8
- net CAM0_C_P: no longer OV5674.9
- net CAM0_D0_N: no longer OV5674.2
- net CAM0_D0_P: no longer OV5674.3
- net CAM0_D1_N: no longer OV5674.5
- net CAM0_D1_P: no longer OV5674.6
- net CAM_GPIO: now also CAMERA.17
- net CDD: now also EINK_524352471.7; no longer J3.7
- net EINK_BUSY: now also C2040.13, EINK_524352471.16; no longer J3.16
- net EINK_CS: now also C2040.16, EINK_524352471.13; no longer J3.13
- net EINK_D/C: now also C2040.15, EINK_524352471.14; no longer J3.14
- net EINK_RESET: now also C2040.14, EINK_524352471.15; no longer J3.15
- net GDR: now also EINK_524352471.23; no longer J3.23
- net GND: now also C24.1, CAMERA.1, CAMERA.10, CAMERA.13, CAMERA.16, CAMERA.19, CAMERA.4, CAMERA.7, EINK_524352471.17, EINK_524352471.8, EINK_524352471.P1, EINK_524352471.P2, FB5.1, JOY_STICK.4, M.2KEYM(NGFF).1, M.2KEYM(NGFF).15, M.2KEYM(NGFF).21, M.2KEYM(NGFF).27, M.2KEYM(NGFF).3, M.2KEYM(NGFF).33, M.2KEYM(NGFF).39, M.2KEYM(NGFF).45, M.2KEYM(NGFF).51, M.2KEYM(NGFF).57, M.2KEYM(NGFF).71, M.2KEYM(NGFF).73, M.2KEYM(NGFF).75, M.2KEYM(NGFF).9, M.2KEYM(NGFF).SH1, M.2KEYM(NGFF).SH2, R19.1, R21.1, U13.8, U5.3, U6.4, U8.3; no longer C24.2, C25.2, C27.2, C28.2, C29.2, C30.2, C31.2, C32.2, C33.2, C34.2, C35.2, C36.2, C37.2, C38.2, C39.2, C41.2, C51.2, C70.2, C78.2, C81.2, FB5.2, GND25.P$1, J3.17, J3.8, J3.P1, J3.P2, OSC1.2, OV5674.1, OV5674.10, OV5674.12, OV5674.21, OV5674.4, OV5674.7, SJ2.1, SJ3.3, SPI_FLASH_SAM.B3, U5.2, U6.2, U7.2, U8.4
- net LEFT_N: now also FB3.2; no longer FB10.2
- net LEFT_P: now also FB2.2; no longer FB9.2
- net N$16: now also Q3.1, U8.4; no longer ANT1.P$2, U8.2
- net N$29: now also FB4.1; no longer FB3.1
- net N$36: now also FB4.2; no longer FB3.2
- net N$40: now also FB2.1; no longer FB9.1
- net N$41: now also FB3.1; no longer FB10.1
- net N$8: now also Q2.1, U5.4; no longer FL5.2, OV5674.16, OV5674.17
- net NC: now also EINK_524352471.24; no longer J3.24
- net OUT: now also FB1.1; no longer FB2.2
- net PREVGH: now also EINK_524352471.4; no longer J3.4
- net PREVGL: now also EINK_524352471.2; no longer J3.2
- net RESE: now also EINK_524352471.22; no longer J3.22
- net SAM_1V1: no longer C78.1
- net SAM_3V3: now also C24.2, JOY_STICK.1, R25.2, R26.2, U5.5, U6.8, U8.5; no longer C70.1, C81.1, SPI_FLASH_SAM.B4
- net SAM_QSPI_SCLK: now also U6.6; no longer SPI_FLASH_SAM.B2
- net SAM_QSPI_SCN: now also U6.1; no longer SPI_FLASH_SAM.C2
- net SAM_QSPI_SD0: now also U6.5; no longer SPI_FLASH_SAM.D3
- net SAM_QSPI_SD1: now also U6.2; no longer SPI_FLASH_SAM.D2
- net SAM_QSPI_SD2: now also U6.3; no longer SPI_FLASH_SAM.C4
- net SAM_QSPI_SD3: now also U6.7; no longer SPI_FLASH_SAM.D4
- net SPI_CLK: now also C2040.17, EINK_524352471.12; no longer J3.12
- net SPI_MOSI: now also C2040.18, EINK_524352471.11; no longer J3.11
- net TSCL: now also EINK_524352471.19; no longer J3.19
- net TSDA: now also EINK_524352471.18; no longer J3.18
- net USB_N: now also U13.5
- net USB_P: now also U13.4
- net VCOM: now also EINK_524352471.1; no longer J3.1
- net VGH: now also EINK_524352471.20; no longer J3.20
- net VGL: now also EINK_524352471.21; no longer J3.21
- net VOUT: now also C26.1
- net VPP: now also EINK_524352471.6; no longer J3.6
- net VSH: now also EINK_524352471.5; no longer J3.5
- net VSL: now also EINK_524352471.3; no longer J3.3
- net V_BATT: no longer C41.1, C51.1
Routing:
- net 3.3V: track 308.1 -> 65.7 mm, vias 19 -> 15
- net SDA: track 201.4 -> 0.00 mm, vias 15 -> 0
- net SCL: track 199.3 -> 0.00 mm, vias 13 -> 0
- net RINPUT1: track 59.4 -> 185.6 mm
- net SAM_SCL: track 0.00 -> 106.1 mm, vias 0 -> 6
- net SAM_SDA: track 0.00 -> 104.0 mm, vias 0 -> 6
- net EINK_CS: track 39.7 -> 130.5 mm, vias 2 -> 3
- net EINK_BUSY: track 49.3 -> 133.9 mm, vias 2 -> 3
- net EINK_RESET: track 49.6 -> 128.3 mm, vias 2 -> 3
- net EINK_D/C: track 47.4 -> 125.7 mm, vias 2 -> 3
- net SPI_CLK: track 42.9 -> 119.8 mm, vias 2 -> 3
- net SPI_MOSI: track 44.9 -> 118.7 mm, vias 2 -> 3
- net VBUS: track 80.3 -> 9.33 mm, vias 4 -> 6
- net PCIE_!RST: track 0.00 -> 69.0 mm, vias 0 -> 4
- net PCIE_CLK_!REQ: track 0.00 -> 67.8 mm, vias 0 -> 4
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- added copper zone on layer 1, net 3.3V
- added copper zone on layer 15, net 3.3V
- added copper zone on layer 15, net 5.0V
- added copper zone on layer 16, net AGND
- added copper zone on layer 1, net BATTERY_IN
- added copper zone on layer 2, net GND
- added copper zone on layer 15, net GND1
- added copper zone on layer 2, net GND2
- added copper zone on layer 1, net GND3
- added copper zone on layer 2, net GND4
- added copper zone on layer 15, net GND5
- added copper zone on layer 16, net GND6
- added copper zone on layer 15, net SAM_3V3
- added copper zone on layer 1, net VBUS
- added copper zone on layer 15, net VBUS
- added copper zone on layer 15, net V_BATT
- removed copper zone on layer 16, net 5.0V
Other:
- board size 66 x 111.6 mm -> 60 x 91 mm
- board text added: "Distiller V1.0 © PamirAI Inc. 2024"
- board text removed: "1V8TP"
- board text removed: "RPIBOOT"
- board text removed: "Reveri H1 V1.0 © PamirAI Inc. 2024"

Commit message: pcb v4
Parts:
- added C25: 100uF, rcl:C1210
- M.2KEYM(NGFF): value 1-2199119-5 -> 1-2199119-5 OR C841645
- U5: value MC74VHC1G14DFT1G -> MC74VHC1G14DFT1G OR C66196
- moved SJ1 5.09 mm to (45.3, 39.4)
- moved C50 5.02 mm to (22.9, 88.0), turned to 180 degrees
- moved R20 3.00 mm to (44.0, 41.6), turned to 90 degrees
- moved R29 1.63 mm to (44.7, 24.3)
- moved C21 1.52 mm to (45.6, 29.9)
- moved R24 1.52 mm to (45.7, 28.6)
- moved R19 1.02 mm to (52.1, 16.2)
- moved LED3 0.51 mm to (29.3, 91.2)
- moved R10 0.51 mm to (31.0, 88.2)
- moved R21 0.51 mm to (52.1, 18.7)
- moved D1 0.51 mm to (31.0, 91.2)
- moved R8 0.51 mm to (29.3, 88.2)
- moved U2 0.51 mm to (33.6, 91.2)
- moved T1 0.47 mm to (40.7, 42.6)
- moved FB3 0.40 mm to (52.2, 22.7)
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Connections:
- net 5.0V: now also C25.1
- net GND: now also C25.2
Routing:
- net ENABLE: track 47.3 -> 39.9 mm, vias 2 -> 3
- net 3.3V: track 65.7 -> 72.6 mm
- net AVDD: track 114.6 -> 108.3 mm
- net GND: track 48.4 -> 54.6 mm, vias 34 -> 211
- net VBUS: track 9.33 -> 5.58 mm
- net N$25: track 18.9 -> 15.5 mm
- net N$2: track 5.17 -> 1.89 mm
- net N_RPIBOOT: track 14.3 -> 17.2 mm
- net N$6: track 2.13 -> 4.41 mm
- net SAM_3V3: track 222.9 -> 220.7 mm
- net RINPUT1: track 185.6 -> 187.0 mm
- net BUTTON_U: track 67.1 -> 68.3 mm
- net !CE!: track 1.63 -> 2.67 mm
- net N$30: track 2.23 -> 1.44 mm
- net SAM_SDA: track 104.0 -> 104.7 mm
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- added copper zone on layer 2, net GND10
- added copper zone on layer 2, net GND7
- added copper zone on layer 15, net GND8
- added copper zone on layer 15, net GND9
Other:
- board size 60 x 91 mm -> 60 x 95 mm
- board text added: "Distiller V0.4 © PamirAI Inc. 2024"
- board text added: "Prototype Build. Sold as is. No warranty expressed or implied. Not approved by the FCC or any other regulatory agency worldwide. Not liable for any direct, indirect, incidental, or consequential damages. Not for critical applications."
- board text removed: "3V3TP"
- board text removed: "5VTP"
- board text removed: "BATT_TP"
- board text removed: "Distiller V1.0 © PamirAI Inc. 2024"
- board text removed: "VOUT_TP"
