File: PCB/AI_EINK.brd (EAGLE design)
At the start: 60 x 95 mm, 161 parts, among them IC3 WM8960, J1 BM04B-GHS-TBT(LF)(SN)(N), J2 C393939, Q1 SI1308EDL-T1-GE3, Q2 NMOS_C7465427, Q3 NMOS_C7465427, T1 MMUN2133LT1G, U1 TPS61092RSAR, U10 AP2112-3.3K, U11 AP2112-3.3K, U12 SPU0410LR5H-QB, U13 TPD4EUSB30DQARDQA10, U2 MC74VHC1G14DFT1G, U3 BQ27441DRZR-G1A, U4 BQ24075, U5 MC74VHC1G14DFT1G OR C66196, U6 W25Q128JVSIQSOIC_128JVSIQ_WIN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, U8 MC74VHC1G14DFT1G, U9 EMC2301-1-ACZL-TRMSOP8_MC_MCH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, Y1 ABM8-272-T3

Commit message: v5 PCB done
Parts:
- removed C52, C54: 33pF, Capacitor:CAPC1005X60
- removed C57: 10uF, Capacitor:CAPC1005X60
- removed FB4: FERRITE_BEAD, Filter:BEADC1608X95N
- added C27: 27pF, Capacitor:CAPC1005X60
- added C29: 4.7uF, Capacitor:CAPC1005X60
- added C30: 1.0uF, Capacitor:CAPC1005X60
- added R27, R37: 10k, Resistor:RESC1005X40
- added R38: 4.7k, Resistor:RESC1005X40
- added R39: 300k, Resistor:RESC1005X40
- added R40, R42: 4.7K, Resistor:RESC1005X40
- added R41: 47K, Resistor:RESC1005X40
- added R43: 10K, Resistor:RESC1005X40
- added R44: 6.57k, Resistor:RESC1005X40
- added SOM_UART: BM04B-GHS-TBT(LF)(SN)(N), BM04B-GHS-TBT_LF__SN__N_:JST_BM04B-GHS-TBT(LF)(SN)(N)
- added U14: OPA344, SparkFun-IC-Amplifiers:SOT23-5
- added USB2.0MUX: TS3USB30RSWR, microbuilder:10-UFQFN
- Q2: value NMOS_C7465427 -> DMG2307L; device Transistor:SOT23 -> DMG2307L:SOT96P240X110-3N
- U12: value SPU0410LR5H-QB -> C233266
- moved RPIBOOT2 42.5 mm to (59.3, 46.3)
- moved GND13 42.5 mm to (59.3, 44.9)
- moved U12 36.9 mm to (58.6, 88.7), turned to 0 degrees
- moved C50 35.8 mm to (58.4, 91.9)
- moved JOY_STICK 3.56 mm to (6.99, 88.8)
- moved U2 2.05 mm to (35.6, 91.4)
- moved LED3 1.61 mm to (30.8, 91.7)
- moved R10 1.61 mm to (32.5, 88.7)
- moved R8 1.61 mm to (30.8, 88.7)
- moved D1 1.61 mm to (32.5, 91.7)
- moved C42 0.92 mm to (23.7, 39.7)
- moved BUS 0.66 mm to (59.3, 54.8)
- moved BUD 0.64 mm to (2.67, 54.4)
- moved BUP 0.64 mm to (2.67, 71.4)
- moved JP6 0.38 mm to (46.5, 8.68)
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Connections:
- removed net N$36: C54.1, C57.1, FB4.2
- removed net N$8: Q2.1, U5.4
- removed net SAM_GPIO1: C2040.3
- removed net SAM_GPIO2: C2040.4
- new net N$10: C29.1, U12.1
- new net N$13: C27.1, R38.1, R39.2, U14.4
- new net N$20: C29.2, R38.2
- new net N$22: C30.1, R27.1, R37.2, U14.3
- new net N$28: Q2.1, R43.2, R44.1
- new net SAM_USB_SWITCH: C2040.30, R41.1, USB2.0MUX.8
- new net UART_RXD0: RPI-CM1.51, SOM_UART.3
- new net UART_RXD3_SAM: C2040.2, R40.1, RPI-CM1.34
- new net UART_TXD0: RPI-CM1.55, SOM_UART.2
- new net UART_TXD3_SAM: C2040.3, R42.1, RPI-CM1.54
- new net USB_SAM_N: R32.1, USB2.0MUX.7
- new net USB_SAM_P: R31.1, USB2.0MUX.1
- net 3.3V: now also Q2.2, R43.1; no longer Q2.3
- net 3V3_EINK: now also Q2.3; no longer Q2.2
- net AVDD: now also R27.2, U14.5
- net EINK_BUSY: now also RPI-CM1.40; no longer RPI-CM1.34
- net GND: now also C30.2, CAMERA.P1, CAMERA.P2, R37.1, R41.2, SOM_UART.4, U14.2, USB2.0MUX.10, USB2.0MUX.4; no longer C52.2, C54.2
- net N$29: now also R44.2, U5.4; no longer C52.1, FB4.1, U12.1
- net RINPUT1: now also C27.2, R39.1, U14.1; no longer C57.2
- net SAM_3V3: now also R40.2, R42.2, USB2.0MUX.9
- net SAM_INTERUPT: now also C2040.4; no longer C2040.2
- net USB_N: now also USB2.0MUX.5; no longer R32.1
- net USB_P: now also USB2.0MUX.3; no longer R31.1
Routing:
- net UART_RXD0: track 0.00 -> 112.0 mm, vias 0 -> 4
- net UART_TXD0: track 0.00 -> 105.2 mm, vias 0 -> 4
- net SAM_USB_SWITCH: track 0.00 -> 89.1 mm, vias 0 -> 6
- net RINPUT1: track 185.7 -> 115.0 mm, vias 2 -> 4
- net USB_SAM_N: track 0.00 -> 64.7 mm, vias 0 -> 2
- net USB_SAM_P: track 0.00 -> 61.8 mm, vias 0 -> 4
- net UART_TXD3_SAM: track 0.00 -> 55.9 mm, vias 0 -> 4
- net UART_RXD3_SAM: track 0.00 -> 47.4 mm, vias 0 -> 4
- net AVDD: track 108.3 -> 148.7 mm, vias 6 -> 9
- net N$10: track 0.00 -> 34.0 mm
- net USB_N: track 153.0 -> 126.4 mm, vias 4 -> 5
- net USB_P: track 152.7 -> 126.4 mm, vias 5 -> 4
- net N$22: track 0.00 -> 14.1 mm, vias 0 -> 2
- net 3.3V: track 72.6 -> 61.9 mm, vias 15 -> 17
- net N$13: track 0.00 -> 10.3 mm
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
Commit message: pcb
Parts:
- removed L2: ASPI-0403S-100M-T, ASPI-0403S-100M-T:IND_ASPI-0403S-100M-T
- added L3: FNR5012S100MT 10uH, LQH5BPN2R2NT0L:IND_LQH5BPN2R2NT0L
- added RPIBOOT3: DNP, SparkFun-Connectors:PAD.03X.03
- CAMERA: value 524372271CON_524372271_MOL -> C262642
- L1: value 6.8uH -> 6.8uH C36410
- LED2: value 5VBOOST -> LED_RED; device microbuilder:CHIPLED_0805_NOOUTLINE -> LED:LEDC1608X65N_RND-R
- LOW_BATT: value XL-2012VRC -> LED_RED; device microbuilder:CHIPLED_0805_NOOUTLINE -> LED:LEDC1608X65N_RND-R
- moved LOW_BATT 0.18 mm to (42.6, 38.9), turned to 90 degrees
- turned LED2 to 90 degrees
Connections:
- net 3V3_EINK: now also L3.1; no longer L2.1
- net EXT_VCC_PCIE: now also RPIBOOT3.P$1
- net N$23: now also L3.2; no longer L2.2
Routing:
- net EXT_VCC_PCIE: track 23.3 -> 27.5 mm
- net 3V3_EINK: track 34.5 -> 33.3 mm
- net GND: vias 180 -> 233
Other:
- board text added: "Distiller V0.5 © PamirAI Inc. 2024"
- board text added: "No warranty expressed or implied. Not for critical applications."
- board text removed: "Distiller V0.4 © PamirAI Inc. 2024"
- board text removed: "Prototype Build. Sold as is. No warranty expressed or implied. Not approved by the FCC or any other regulatory agency worldwide. Not liable for any direct, indirect, incidental, or consequential damages. Not for critical applications."

Commit message: pcb
Parts:
- removed JOY_STICK, SOM_UART: BM04B-GHS-TBT(LF)(SN)(N), BM04B-GHS-TBT_LF__SN__N_:JST_BM04B-GHS-TBT(LF)(SN)(N)
- removed JP6: S2B-PH-SM4-TB, SparkFun-Connectors:JST-2-SMD
- removed R29: 10K, Resistor:RESC1005X40
- removed U8: MC74VHC1G14DFT1G, MC74VHC1G14DFT1G:SOT65P210X110-5N
- added C28, C32, C33, C36: 10uF, Capacitor:CAPC1005X60
- added C31: 0.1uF, Capacitor:CAPC1005X60
- added C34, C35: 1uF, Capacitor:CAPC1005X60
- added GND36, GND37, GND40, GND41, GND42, GND7, RPIBOOT10, RPIBOOT11, RPIBOOT12, RPIBOOT6, RPIBOOT8, RPIBOOT9: DNP, SparkFun-Connectors:PAD.03X.03
- added H2, J3, J4, J5: BM04B-SRSS-TBCONN4_BM04B-SRSS_JST, 2024-05-18_10-24-10_Library:CONN4_BM04B-SRSS_JST
- added IC1: LIS3MDL, adafruit_sensor:LGA12_2X2MM
- added Q4: NMOS_C7465427, Transistor:SOT23
- added RPIBOOT7: TEST-POINT3, SparkFun-Connectors:PAD.03X.03
- added U15: AP2112-3.3K, microbuilder:SOT23-5
- added U16: W25Q16JVUXIQ_TR, W25Q16JVUXIQ_TR:PSON50P300X200X60-9N
- added U17, U18, U19, U20, U21, U22, U23, U24: TPD1E1B04DPYRDPY2_TEX, 2024-05-19_00-17-33_Library:DPY2_TEX
- added U25: DRV2605LDGSR, DRV2605LDGSR:SOP50P490X110-10N
- added U7: SN74LVC244ARWPRRWP0020A, 2024-05-18_09-46-26_Library:RWP0020A
- J1: value BM04B-GHS-TBT(LF)(SN)(N) -> SM03B-SRSS-TBCONN_SM03B-SRSS-TB_JST; device BM04B-GHS-TBT_LF__SN__N_:JST_BM04B-GHS-TBT(LF)(SN)(N) -> 2024-05-21_05-27-43_Library:CONN_SM03B-SRSS-TB_JST
- R39: value 300k -> 10k
- U6: value W25Q128JVSIQSOIC_128JVSIQ_WIN-L -> LSM6DS3; device 2024-03-29_04-43-21_Library:SOIC_128JVSIQ_WIN-L -> adafruit_sensor:LGA-14L
- moved GND22 54.6 mm to (18.4, 61.7), flipped to the bottom
- moved J1 34.3 mm to (46.6, 11.3), turned to 0 degrees
- moved SJ1 15.0 mm to (44.8, 24.4), turned to 0 degrees
- moved GND27 10.5 mm to (9.92, 2.98)
- moved GND26 9.09 mm to (8.28, 2.98)
- moved C65 5.34 mm to (3.01, 6.79)
- moved R11 5.26 mm to (41.6, 12.5), turned to 270 degrees
- moved U6 4.95 mm to (21.8, 44.2)
- moved C66 4.58 mm to (3.01, 13.1)
- moved U10 4.58 mm to (4.19, 10.3)
- moved C67 4.58 mm to (3.04, 14.8)
- moved C68 4.58 mm to (3.04, 16.0)
- moved FB1 4.58 mm to (5.21, 13.1)
- moved FB5 4.58 mm to (5.21, 14.7)
- moved C24 4.34 mm to (21.3, 40.0), turned to 0 degrees
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Connections:
- net SAM_EINK_ON renamed SAM_EINK_PWR
- removed net N$25: R29.1, SJ1.2
- removed net SAM_GPIO22: C2040.34
- removed net SAM_GPIO25: C2040.37
- new net 2A3: U7.14
- new net 2A4: U7.16
- new net 2Y3: U7.4
- new net 2Y4: U7.2
- new net HAP_3V3: C33.1, C35.1, U15.5, U25.10, U25.5, U25.6
- new net N$8: C31.1, IC1.4
- new net SAM_BOOT: Q4.1, RPI-CM1.29
- new net SAM_EINK_SWITCH: C2040.34, U7.18, U7.20
- new net SAM_GPIO23: C2040.35
- new net SOC_EINK_BUSY: RPI-CM1.40, U7.17
- new net SOC_EINK_CS: RPI-CM1.39, U7.7
- new net SOC_EINK_D/C: RPI-CM1.30, U7.5
- new net SOC_EINK_RESET: RPI-CM1.28, U7.3
- new net SOC_SPI_CLK: RPI-CM1.38, U7.10
- new net SOC_SPI_MOSI: RPI-CM1.44, U7.12
- new net THERM: J1.2, SJ1.1
- new net U25_OUT+: H2.1, H2.2, U25.7
- new net U25_OUT-: H2.3, H2.4, U25.9
- net 3.3V: now also C28.1, C36.2, IC1.5, IC1.6, U6.5, U6.8; no longer C7.1, Q2.2, R43.1
- net 5.0V: now also J3.3; no longer J1.3
- net BATTERY_IN: now also J1.3; no longer JP6.2
- net EINK_BUSY: now also RPIBOOT9.P$1, U18.2, U7.1; no longer RPI-CM1.40
- net EINK_CS: now also GND41.P$1, U20.2, U7.11; no longer RPI-CM1.39
- net EINK_D/C: now also RPIBOOT10.P$1, U19.2, U7.13; no longer RPI-CM1.30
- net EINK_RESET: now also GND40.P$1, U17.2, U7.15; no longer RPI-CM1.28
- net FAN_PWM: now also J3.1; no longer J1.1
- net GND: now also C28.2, C31.2, C32.2, C33.2, C34.1, C35.2, C36.1, IC1.12, IC1.2, IC1.3, IC1.9, J1.1, J3.4, J4.4, J5.3, J5.4, Q4.2, U15.2, U16.4, U17.1, U18.1, U19.1, U20.1, U21.1, U22.1, U23.1, U24.1, U25.4, U25.8, U6.1, U6.6, U6.7, U7.21, U7.9; no longer J1.4, J1.S1, J1.S2, JOY_STICK.4, JP6.1, SJ1.1, SOM_UART.4, U6.4, U8.3
- net N$16: now also C34.2, U25.1; no longer Q3.1, U8.4
- net N$24: now also Q4.3
- net SAM_3V3: now also C7.1, J4.1, Q2.2, R43.1, U16.8, U7.19; no longer JOY_STICK.1, U6.8, U8.5
- net SAM_INTERUPT: now also RPIBOOT12.P$1
- net SAM_QSPI_SCLK: now also U16.6; no longer U6.6
- net SAM_QSPI_SCN: now also U16.1; no longer U6.1
- net SAM_QSPI_SD0: now also U16.5; no longer U6.5
- net SAM_QSPI_SD1: now also U16.2; no longer U6.2
- net SAM_QSPI_SD2: now also U16.3; no longer U6.3
- net SAM_QSPI_SD3: now also U16.7; no longer U6.7
- net SAM_SCL: now also C2040.37, J4.3, RPIBOOT8.P$1, U25.2; no longer C2040.35, JOY_STICK.3
- net SAM_SDA: now also GND37.P$1, J4.2, U25.3; no longer JOY_STICK.2
- net SCL1: now also IC1.1, RPIBOOT6.P$1, U6.13
- net SDA1: now also GND7.P$1, IC1.11, U6.14
- net SPI_CLK: now also RPIBOOT11.P$1, U21.2, U7.8; no longer RPI-CM1.38
- net SPI_MOSI: now also GND42.P$1, U22.2, U7.6; no longer RPI-CM1.44
- net SYS_PI_ON: now also Q3.1; no longer U8.2
- net TACH: now also J3.2; no longer J1.2
- net TS: now also SJ1.2; no longer R29.2
- net TSCL: now also U23.2
- net TSDA: now also U24.2
- net UART_RXD0: now also J5.2; no longer SOM_UART.3
- net UART_RXD3_SAM: now also RPIBOOT7.P$1
- net UART_TXD0: now also J5.1; no longer SOM_UART.2
- net UART_TXD3_SAM: now also GND36.P$1
- net VOUT: now also C32.1, U15.1, U15.3
Routing:
- net VOUT: track 65.1 -> 159.9 mm, vias 5 -> 7
- net SOC_EINK_CS: track 0.00 -> 85.7 mm, vias 0 -> 4
- net SOC_SPI_MOSI: track 0.00 -> 82.0 mm, vias 0 -> 3
- net SOC_SPI_CLK: track 0.00 -> 81.8 mm, vias 0 -> 3
- net SOC_EINK_BUSY: track 0.00 -> 78.8 mm, vias 0 -> 3
- net SOC_EINK_D/C: track 0.00 -> 75.1 mm, vias 0 -> 2
- net SOC_EINK_RESET: track 0.00 -> 74.0 mm, vias 0 -> 2
- net EINK_CS: track 130.3 -> 64.0 mm
- net EINK_BUSY: track 134.2 -> 70.6 mm, vias 3 -> 4
- net EINK_D/C: track 126.1 -> 68.1 mm
- net EINK_RESET: track 128.5 -> 70.9 mm
- net SPI_CLK: track 119.0 -> 65.9 mm, vias 3 -> 4
- net SPI_MOSI: track 118.0 -> 69.5 mm, vias 3 -> 4
- net SAM_EINK_SWITCH: track 0.00 -> 24.4 mm, vias 0 -> 4
- net SCL1: track 52.4 -> 76.4 mm, vias 3 -> 4
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Other:
- board text added: "Distiller V0.6 © PamirAI Inc. 2024"
- board text removed: "Distiller V0.5 © PamirAI Inc. 2024"

Commit message: v0.7
Parts:
- removed J3: BM04B-SRSS-TBCONN4_BM04B-SRSS_JST, 2024-05-18_10-24-10_Library:CONN4_BM04B-SRSS_JST
- added J6: SM04B-SRSS-TBCONN_SM04B-SRSS-TB_JST, 2024-06-16_01-36-12_Library:CONN_SM04B-SRSS-TB_JST
- moved C42 0.23 mm to (23.5, 39.6)
Connections:
- net 5.0V: now also J6.3; no longer J3.3
- net FAN_PWM: now also J6.1; no longer J3.1
- net GND: now also J6.4; no longer J3.4
- net TACH: now also J6.2; no longer J3.2
Routing:
- net 5.0V: track 100.9 -> 104.5 mm
- net FAN_PWM: track 16.3 -> 17.0 mm
- net SAM_SDA: track 116.1 -> 115.6 mm
- net I2S_DIN: track 43.6 -> 44.1 mm, vias 2 -> 3
- net TACH: track 21.6 -> 21.9 mm, vias 3 -> 2
- net I2S_DOUT: track 45.9 -> 45.7 mm, vias 2 -> 3
- net GND: track 83.9 -> 84.0 mm, vias 253 -> 258
Other:
- board text added: "Distiller V0.7 © PamirAI Inc. 2024"
- board text removed: "Distiller V0.6 © PamirAI Inc. 2024"

Commit message: before modification, v0.7, for fateen and adam
Changed lines of the file:
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@@
 <drawing>
 <settings>
-<setting alwaysvectorfont="yes"/>
+<setting alwaysvectorfont="no"/>
 <setting verticaltext="up"/>
 </settings>
@@
 <via x="29.083" y="26.543" extent="1-16" drill="0.3"/>
 <wire x1="29.083" y1="26.829575" x2="27.178" y2="28.734575" width="0.0889" layer="1"/>
-<wire x1="43.3346" y1="21.3815" x2="42.8139" y2="21.3815" width="0.0889" layer="1"/>
-<wire x1="42.8139" y1="21.3815" x2="42.5546" y2="21.6408" width="0.0889" layer="1"/>
-<wire x1="42.5546" y1="21.6408" x2="36.3982" y2="21.6408" width="0.0889" layer="1"/>
-<wire x1="36.3982" y1="21.6408" x2="35.941" y2="22.098" width="0.0889" layer="1"/>
+<wire x1="43.3346" y1="21.3815" x2="36.6575" y2="21.3815" width="0.0889" layer="1"/>
+<wire x1="36.6575" y1="21.3815" x2="35.941" y2="22.098" width="0.0889" layer="1"/>
 <via x="35.941" y="22.098" extent="1-16" drill="0.3"/>
 <wire x1="41.867" y1="87.797" x2="40.684" y2="86.614" width="0.2032" layer="1"/>

Commit message: ESP32
Parts:
- added C37, C38: 0.1uF, Capacitor:CAPC1005X60
- added C39, C54, C55: 10uF, Capacitor:CAPC1005X60
- added C52, C57: 220pF, Capacitor:CAPC1005X60
- added DISPLAY: C262642, 2024-03-29_02-21-27_Library:CON_524372271_MOL
- added FB4, FB7: 120o, Filter:BEADC1608X95N
- added J10, J11, J8, J9: SM04B-SRSS-TBCONN_SM04B-SRSS-TB_JST, 2024-06-16_01-36-12_Library:CONN_SM04B-SRSS-TB_JST
- added J3, J7: SM02B-SRSS-TB(LF)(SN), SM02B-SRSS-TB_LF__SN_:SM02B-SRSS-TB(LF)(SN)
- added R29: 8.2k, Resistor:RESC1005X40
- added R46: 10K Trim, adafruit_electromech:RTRIM3314J
- added R48, R49: 30k, Resistor:RESC1005X40
- added U$120, U$123: MOUNTINGHOLE2.5, microbuilder:MOUNTINGHOLE_2.5_PLATED
- added U8: PAM8302, microbuilder:MSOP8_0.65MM
- moved J4 4.70 mm to (9.53, 89.9), flipped to the bottom, turned to 270 degrees
- moved C46 1.02 mm to (9.64, 6.41)
- moved C48 1.02 mm to (8.24, 6.41)
Connections:
- net N$11 renamed PI_PWR_INDICATE
- removed net N$40: FB2.1, IC3.25
- removed net N$41: FB3.1, IC3.23
- removed net N$6: R20.2, T1.C
- new net IN+: R48.2, U8.3
- new net IN-: R49.2, U8.4
- new net LINPUT1: IC3.4, J7.2
- new net LOW_BATT_P: J10.3, R20.2, T1.C
- new net N$25: C38.2, R49.1
- new net N$31: C37.2, R48.1
- new net N$32: C37.1, R29.2, R46.3
- new net OUT+: FB7.1, U8.5
- new net OUT-: FB4.1, U8.8
- new net SPK_LN: C38.1, FB3.1, IC3.23, R46.1
- new net SPK_LP: FB2.1, IC3.25, R29.1
- new net SPK_RN: IC3.19
- new net SPK_RP: IC3.22
- new net VO+: C57.1, FB7.2, J3.1
- new net VO-: C52.1, FB4.2, J3.2
- net !CHG!: now also J10.2
- net 3.3V: now also DISPLAY.22
- net 5.0V: now also C39.1, C54.1, C55.1, U8.1, U8.6
- net BUTTON_D: now also J11.3
- net BUTTON_U: now also J11.2
- net DSI1_C_N: now also DISPLAY.8
- net DSI1_C_P: now also DISPLAY.9
- net DSI1_D0_N: now also DISPLAY.2
- net DSI1_D0_P: now also DISPLAY.3
- net DSI1_D1_N: now also DISPLAY.5
- net DSI1_D1_P: now also DISPLAY.6
- net DSI1_D2_N: now also DISPLAY.11
- net DSI1_D2_P: now also DISPLAY.12
- net DSI1_D3_N: now also DISPLAY.14
- net DSI1_D3_P: now also DISPLAY.15
- net GND: now also C39.2, C52.2, C54.2, C55.2, C57.2, DISPLAY.1, DISPLAY.10, DISPLAY.13, DISPLAY.16, DISPLAY.19, DISPLAY.4, DISPLAY.7, DISPLAY.P1, DISPLAY.P2, J10.4, J11.4, J7.1, J8.3, J8.4, J9.4, U8.7
- net SAM_3V3: now also J11.1
- net SCL0: now also DISPLAY.20
- net SDA0: now also DISPLAY.21
- net USB_N: now also J9.3
- net USB_P: now also J9.2
- net VBUS: now also J8.1, J8.2, J9.1
- net VOUT: now also J10.1
Routing:
- net SPK_LP: track 0.00 -> 110.9 mm, vias 0 -> 4
- net N$40: track 98.0 -> 0.00 mm, vias 4 -> 0
- net LINPUT1: track 0.00 -> 91.9 mm, vias 0 -> 4
- net SPK_LN: track 0.00 -> 90.5 mm, vias 0 -> 2
- net N$41: track 71.5 -> 0.00 mm, vias 2 -> 0
- net 5.0V: track 104.5 -> 141.9 mm, vias 13 -> 17
- net LOW_BATT_P: track 0.00 -> 27.2 mm, vias 0 -> 1
- net SDA0: track 38.2 -> 60.1 mm
- net SCL0: track 39.4 -> 58.2 mm
- net GND: track 84.0 -> 102.4 mm, vias 258 -> 254
- net BUTTON_D: track 50.4 -> 62.2 mm
- net DSI1_D3_P: track 0.00 -> 11.5 mm, vias 0 -> 2
- net OUT-: track 0.00 -> 11.0 mm, vias 0 -> 2
- net DSI1_D3_N: track 0.00 -> 10.8 mm, vias 0 -> 2
- net DSI1_C_N: track 0.00 -> 10.7 mm, vias 0 -> 1
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- removed copper zone on layer 16, net GND6
Other:
- board text added: "Distiller Type A V0.1 © PamirAI Inc. 2024"
- board text added: "MIPI DISPLAY"
- board text added: "POWER LEDS"
- board text added: "POWER SUPPLY"
- board text added: "SAM GPIO"
- board text added: "SAM I2C"
- board text added: "USB2.0"
- board text removed: "Distiller V0.7 © PamirAI Inc. 2024"
- board text removed: "EINK"
